Commit message: final

File: bodies/body1.urdf (robot description, URDF)
Before this commit: robot robot, 5 links, 4 joints
Links:
- link m: geometry collision box size=1 6 0.5; visual box size=1 6 0.5
Joints:
- joint m_L0: origin xyz=-0.5 -2.5 1 rpy=0 0 0 -> xyz=-0.5 -3.0 1 rpy=0 0 0
- joint m_r0: origin xyz=0.5 -2.5 1 rpy=0 0 0 -> xyz=0.5 -3.0 1 rpy=0 0 0

File: bodies/body2.urdf (robot description, URDF)
Before this commit: robot robot, 17 links, 16 joints
Links:
- removed link L1
- removed link L2
- removed link LL1
- removed link LL2
- removed link r1
- removed link r2
- removed link r3
- removed link r4
- removed link rl1
- removed link rl2
- removed link rl3
- removed link rl4
- link m: geometry collision box size=1 6 0.5; visual box size=1 6 0.5
Joints:
- removed joint L1_LL1
- removed joint L2_LL2
- removed joint m_L1
- removed joint m_L2
- removed joint m_r1
- removed joint m_r2
- removed joint m_r3
- removed joint m_r4
- removed joint r1_rl1
- removed joint r2_rl2
- removed joint r3_rl3
- removed joint r4_rl4
- joint m_L0: origin xyz=-0.5 -2.5 1 rpy=0 0 0 -> xyz=-0.5 -3.0 1 rpy=0 0 0
- joint m_r0: origin xyz=0.5 -2.5 1 rpy=0 0 0 -> xyz=0.5 -3.0 1 rpy=0 0 0

File: bodies/body3.urdf (robot description, URDF)
Before this commit: robot robot, 15 links, 14 joints
Links:
- removed link L1
- removed link L2
- removed link L3
- removed link LL1
- removed link LL2
- removed link LL3
- removed link r1
- removed link r2
- removed link rl1
- removed link rl2
Joints:
- removed joint L1_LL1
- removed joint L2_LL2
- removed joint L3_LL3
- removed joint m_L1
- removed joint m_L2
- removed joint m_L3
- removed joint m_r1
- removed joint m_r2
- removed joint r1_rl1
- removed joint r2_rl2

File: bodies/body4.urdf (robot description, URDF)
Before this commit: robot robot, 13 links, 12 joints
Links:
- removed link r1
- removed link r2
- removed link r3
- removed link r4
- removed link rl1
- removed link rl2
- removed link rl3
- removed link rl4
- link m: geometry collision box size=1 6 0.5; visual box size=1 6 0.5
Joints:
- removed joint m_r1
- removed joint m_r2
- removed joint m_r3
- removed joint m_r4
- removed joint r1_rl1
- removed joint r2_rl2
- removed joint r3_rl3
- removed joint r4_rl4
- joint m_L0: origin xyz=-0.5 -1.5 1 rpy=0 0 0 -> xyz=-0.5 -3.0 1 rpy=0 0 0
- joint m_r0: origin xyz=0.5 -1.5 1 rpy=0 0 0 -> xyz=0.5 -3.0 1 rpy=0 0 0

File: bodies/body5.urdf (robot description, URDF)
Before this commit: robot robot, 11 links, 10 joints
Links:
- removed link L1
- removed link L2
- removed link LL1
- removed link LL2
- removed link r1
- removed link rl1
- link m: geometry collision box size=1 6 0.5; visual box size=1 6 0.5
Joints:
- removed joint L1_LL1
- removed joint L2_LL2
- removed joint m_L1
- removed joint m_L2
- removed joint m_r1
- removed joint r1_rl1
- joint m_L0: origin xyz=-0.5 -1.5 1 rpy=0 0 0 -> xyz=-0.5 -3.0 1 rpy=0 0 0
- joint m_r0: origin xyz=0.5 -1.5 1 rpy=0 0 0 -> xyz=0.5 -3.0 1 rpy=0 0 0

File: bodies/body6.urdf (robot description, URDF)
Before this commit: robot robot, 9 links, 8 joints
Links:
- removed link L1
- removed link LL1
- removed link r1
- removed link rl1
- link m: geometry collision box size=1 6 0.5; visual box size=1 6 0.5
Joints:
- removed joint L1_LL1
- removed joint m_L1
- removed joint m_r1
- removed joint r1_rl1
- joint m_L0: origin xyz=-0.5 -1.5 1 rpy=0 0 0 -> xyz=-0.5 -3.0 1 rpy=0 0 0
- joint m_r0: origin xyz=0.5 -1.5 1 rpy=0 0 0 -> xyz=0.5 -3.0 1 rpy=0 0 0

File: bodies/body7.urdf (robot description, URDF)
Before this commit: robot robot, 11 links, 10 joints
Links:
- removed link r1
- removed link r2
- removed link r3
- removed link rl1
- removed link rl2
- removed link rl3
- link m: geometry collision box size=1 6 0.5; visual box size=1 6 0.5
Joints:
- removed joint m_r1
- removed joint m_r2
- removed joint m_r3
- removed joint r1_rl1
- removed joint r2_rl2
- removed joint r3_rl3
- joint m_L0: origin xyz=-0.5 -4.0 1 rpy=0 0 0 -> xyz=-0.5 -3.0 1 rpy=0 0 0
- joint m_r0: origin xyz=0.5 -4.0 1 rpy=0 0 0 -> xyz=0.5 -3.0 1 rpy=0 0 0

File: bodies/body8.urdf (robot description, URDF)
Before this commit: robot robot, 19 links, 18 joints
Links:
- removed link L1
- removed link L2
- removed link L3
- removed link L4
- removed link LL1
- removed link LL2
- removed link LL3
- removed link LL4
- removed link r1
- removed link r2
- removed link r3
- removed link rl1
- removed link rl2
- removed link rl3
Joints:
- removed joint L1_LL1
- removed joint L2_LL2
- removed joint L3_LL3
- removed joint L4_LL4
- removed joint m_L1
- removed joint m_L2
- removed joint m_L3
- removed joint m_L4
- removed joint m_r1
- removed joint m_r2
- removed joint m_r3
- removed joint r1_rl1
- removed joint r2_rl2
- removed joint r3_rl3

File: bodies/body9.urdf (robot description, URDF)
Before this commit: robot robot, 13 links, 12 joints
Links:
- removed link L1
- removed link LL1
- removed link r1
- removed link r2
- removed link r3
- removed link rl1
- removed link rl2
- removed link rl3
- link m: geometry collision box size=1 6 0.5; visual box size=1 6 0.5
Joints:
- removed joint L1_LL1
- removed joint m_L1
- removed joint m_r1
- removed joint m_r2
- removed joint m_r3
- removed joint r1_rl1
- removed joint r2_rl2
- removed joint r3_rl3
- joint m_L0: origin xyz=-0.5 -1.5 1 rpy=0 0 0 -> xyz=-0.5 -3.0 1 rpy=0 0 0
- joint m_r0: origin xyz=0.5 -1.5 1 rpy=0 0 0 -> xyz=0.5 -3.0 1 rpy=0 0 0
