Commit message: milliped

File: bodies/body0.urdf (robot description, URDF)
Before this commit: robot robot, 15 links, 14 joints
Links:
- removed link r1
- removed link r2
- removed link r3
- removed link rl1
- removed link rl2
- removed link rl3
Joints:
- removed joint m_r1
- removed joint m_r2
- removed joint m_r3
- removed joint r1_rl1
- removed joint r2_rl2
- removed joint r3_rl3

File: bodies/body2.urdf (robot description, URDF)
Before this commit: robot robot, 15 links, 14 joints
Links:
- added link r4, mass 1; collision box size=1 0.2 0.2; visual box size=1 0.2 0.2
- added link rl4, mass 1; collision box size=0.2 0.2 1; visual box size=0.2 0.2 1
- link m: geometry collision box size=1 5 0.5; visual box size=1 5 0.5
Joints:
- added joint m_r4: type revolute, parent m, child r4, origin xyz=0.5 2.3 1 rpy=0 0 0, axis 1 0 0, limit lower=-3.14159 upper=3.14159 effort=0.0 velocity=0.0
- added joint r4_rl4: type revolute, parent r4, child rl4, origin xyz=1 0 0 rpy=0 0 0, axis 1 0 0, limit lower=-3.14159 upper=3.14159 effort=0.0 velocity=0.0
- joint m_L0: origin xyz=-0.5 -3.0 1 rpy=0 0 0 -> xyz=-0.5 -2.5 1 rpy=0 0 0
- joint m_L1: origin xyz=-0.5 -0.6666666666666665 1 rpy=0 0 0 -> xyz=-0.5 -0.5 1 rpy=0 0 0
- joint m_L2: origin xyz=-0.5 1.666666666666667 1 rpy=0 0 0 -> xyz=-0.5 1.5 1 rpy=0 0 0
- joint m_r0: origin xyz=0.5 -3.0 1 rpy=0 0 0 -> xyz=0.5 -2.5 1 rpy=0 0 0
- joint m_r1: origin xyz=0.5 -1.25 1 rpy=0 0 0 -> xyz=0.5 -1.3 1 rpy=0 0 0
- joint m_r2: origin xyz=0.5 0.5 1 rpy=0 0 0 -> xyz=0.5 -0.10000000000000009 1 rpy=0 0 0
- joint m_r3: origin xyz=0.5 2.25 1 rpy=0 0 0 -> xyz=0.5 1.0999999999999996 1 rpy=0 0 0

File: bodies/body3.urdf (robot description, URDF)
Before this commit: robot robot, 15 links, 14 joints
Links:
- removed link r3
- removed link rl3
- added link L3, mass 1; collision box size=1 0.2 0.2; visual box size=1 0.2 0.2
- added link LL3, mass 1; collision box size=0.2 0.2 1; visual box size=0.2 0.2 1
Joints:
- removed joint m_r3
- removed joint r3_rl3
- added joint L3_LL3: type revolute, parent L3, child LL3, origin xyz=-1 0 0 rpy=0 0 0, axis 1 0 0, limit lower=-3.14159 upper=3.14159 effort=0.0 velocity=0.0
- added joint m_L3: type revolute, parent m, child L3, origin xyz=-0.5 2.25 1 rpy=0 0 0, axis 1 0 0, limit lower=-3.14159 upper=3.14159 effort=0.0 velocity=0.0
- joint m_L1: origin xyz=-0.5 -0.6666666666666665 1 rpy=0 0 0 -> xyz=-0.5 -1.25 1 rpy=0 0 0
- joint m_L2: origin xyz=-0.5 1.666666666666667 1 rpy=0 0 0 -> xyz=-0.5 0.5 1 rpy=0 0 0
- joint m_r1: origin xyz=0.5 -1.25 1 rpy=0 0 0 -> xyz=0.5 -0.6666666666666665 1 rpy=0 0 0
- joint m_r2: origin xyz=0.5 0.5 1 rpy=0 0 0 -> xyz=0.5 1.666666666666667 1 rpy=0 0 0

File: bodies/body4.urdf (robot description, URDF)
Before this commit: robot robot, 15 links, 14 joints
Links:
- removed link L1
- removed link L2
- removed link LL1
- removed link LL2
- added link r4, mass 1; collision box size=1 0.2 0.2; visual box size=1 0.2 0.2
- added link rl4, mass 1; collision box size=0.2 0.2 1; visual box size=0.2 0.2 1
- link m: geometry collision box size=1 3 0.5; visual box size=1 3 0.5
Joints:
- removed joint L1_LL1
- removed joint L2_LL2
- removed joint m_L1
- removed joint m_L2
- added joint m_r4: type revolute, parent m, child r4, origin xyz=0.5 1.7000000000000002 1 rpy=0 0 0, axis 1 0 0, limit lower=-3.14159 upper=3.14159 effort=0.0 velocity=0.0
- added joint r4_rl4: type revolute, parent r4, child rl4, origin xyz=1 0 0 rpy=0 0 0, axis 1 0 0, limit lower=-3.14159 upper=3.14159 effort=0.0 velocity=0.0
- joint m_L0: origin xyz=-0.5 -3.0 1 rpy=0 0 0 -> xyz=-0.5 -1.5 1 rpy=0 0 0
- joint m_r0: origin xyz=0.5 -3.0 1 rpy=0 0 0 -> xyz=0.5 -1.5 1 rpy=0 0 0
- joint m_r1: origin xyz=0.5 -1.25 1 rpy=0 0 0 -> xyz=0.5 -0.7 1 rpy=0 0 0
- joint m_r2: origin xyz=0.5 0.5 1 rpy=0 0 0 -> xyz=0.5 0.10000000000000009 1 rpy=0 0 0
- joint m_r3: origin xyz=0.5 2.25 1 rpy=0 0 0 -> xyz=0.5 0.9000000000000004 1 rpy=0 0 0

File: bodies/body5.urdf (robot description, URDF)
Before this commit: robot robot, 15 links, 14 joints
Links:
- removed link r2
- removed link r3
- removed link rl2
- removed link rl3
- link m: geometry collision box size=1 3 0.5; visual box size=1 3 0.5
Joints:
- removed joint m_r2
- removed joint m_r3
- removed joint r2_rl2
- removed joint r3_rl3
- joint m_L0: origin xyz=-0.5 -3.0 1 rpy=0 0 0 -> xyz=-0.5 -1.5 1 rpy=0 0 0
- joint m_L1: origin xyz=-0.5 -0.6666666666666665 1 rpy=0 0 0 -> xyz=-0.5 -0.16666666666666674 1 rpy=0 0 0
- joint m_L2: origin xyz=-0.5 1.666666666666667 1 rpy=0 0 0 -> xyz=-0.5 1.1666666666666665 1 rpy=0 0 0
- joint m_r0: origin xyz=0.5 -3.0 1 rpy=0 0 0 -> xyz=0.5 -1.5 1 rpy=0 0 0
- joint m_r1: origin xyz=0.5 -1.25 1 rpy=0 0 0 -> xyz=0.5 0.5 1 rpy=0 0 0

File: bodies/body6.urdf (robot description, URDF)
Before this commit: robot robot, 15 links, 14 joints
Links:
- removed link L2
- removed link LL2
- removed link r2
- removed link r3
- removed link rl2
- removed link rl3
- link m: geometry collision box size=1 3 0.5; visual box size=1 3 0.5
Joints:
- removed joint L2_LL2
- removed joint m_L2
- removed joint m_r2
- removed joint m_r3
- removed joint r2_rl2
- removed joint r3_rl3
- joint m_L0: origin xyz=-0.5 -3.0 1 rpy=0 0 0 -> xyz=-0.5 -1.5 1 rpy=0 0 0
- joint m_L1: origin xyz=-0.5 -0.6666666666666665 1 rpy=0 0 0 -> xyz=-0.5 0.5 1 rpy=0 0 0
- joint m_r0: origin xyz=0.5 -3.0 1 rpy=0 0 0 -> xyz=0.5 -1.5 1 rpy=0 0 0
- joint m_r1: origin xyz=0.5 -1.25 1 rpy=0 0 0 -> xyz=0.5 0.5 1 rpy=0 0 0

File: bodies/body7.urdf (robot description, URDF)
Before this commit: robot robot, 15 links, 14 joints
Links:
- removed link L1
- removed link L2
- removed link LL1
- removed link LL2
- link m: geometry collision box size=1 8 0.5; visual box size=1 8 0.5
Joints:
- removed joint L1_LL1
- removed joint L2_LL2
- removed joint m_L1
- removed joint m_L2
- joint m_L0: origin xyz=-0.5 -3.0 1 rpy=0 0 0 -> xyz=-0.5 -4.0 1 rpy=0 0 0
- joint m_r0: origin xyz=0.5 -3.0 1 rpy=0 0 0 -> xyz=0.5 -4.0 1 rpy=0 0 0
- joint m_r1: origin xyz=0.5 -1.25 1 rpy=0 0 0 -> xyz=0.5 -1.75 1 rpy=0 0 0
- joint m_r3: origin xyz=0.5 2.25 1 rpy=0 0 0 -> xyz=0.5 2.75 1 rpy=0 0 0

File: bodies/body8.urdf (robot description, URDF)
Before this commit: robot robot, 15 links, 14 joints
Links:
- added link L3, mass 1; collision box size=1 0.2 0.2; visual box size=1 0.2 0.2
- added link L4, mass 1; collision box size=1 0.2 0.2; visual box size=1 0.2 0.2
- added link LL3, mass 1; collision box size=0.2 0.2 1; visual box size=0.2 0.2 1
- added link LL4, mass 1; collision box size=0.2 0.2 1; visual box size=0.2 0.2 1
Joints:
- added joint L3_LL3: type revolute, parent L3, child LL3, origin xyz=-1 0 0 rpy=0 0 0, axis 1 0 0, limit lower=-3.14159 upper=3.14159 effort=0.0 velocity=0.0
- added joint L4_LL4: type revolute, parent L4, child LL4, origin xyz=-1 0 0 rpy=0 0 0, axis 1 0 0, limit lower=-3.14159 upper=3.14159 effort=0.0 velocity=0.0
- added joint m_L3: type revolute, parent m, child L3, origin xyz=-0.5 1.1999999999999993 1 rpy=0 0 0, axis 1 0 0, limit lower=-3.14159 upper=3.14159 effort=0.0 velocity=0.0
- added joint m_L4: type revolute, parent m, child L4, origin xyz=-0.5 2.5999999999999996 1 rpy=0 0 0, axis 1 0 0, limit lower=-3.14159 upper=3.14159 effort=0.0 velocity=0.0
- joint m_L1: origin xyz=-0.5 -0.6666666666666665 1 rpy=0 0 0 -> xyz=-0.5 -1.6 1 rpy=0 0 0
- joint m_L2: origin xyz=-0.5 1.666666666666667 1 rpy=0 0 0 -> xyz=-0.5 -0.20000000000000018 1 rpy=0 0 0

File: bodies/body9.urdf (robot description, URDF)
Before this commit: robot robot, 15 links, 14 joints
Links:
- removed link L2
- removed link LL2
- link m: geometry collision box size=1 3 0.5; visual box size=1 3 0.5
Joints:
- removed joint L2_LL2
- removed joint m_L2
- joint m_L0: origin xyz=-0.5 -3.0 1 rpy=0 0 0 -> xyz=-0.5 -1.5 1 rpy=0 0 0
- joint m_L1: origin xyz=-0.5 -0.6666666666666665 1 rpy=0 0 0 -> xyz=-0.5 0.5 1 rpy=0 0 0
- joint m_r0: origin xyz=0.5 -3.0 1 rpy=0 0 0 -> xyz=0.5 -1.5 1 rpy=0 0 0
- joint m_r1: origin xyz=0.5 -1.25 1 rpy=0 0 0 -> xyz=0.5 -0.5 1 rpy=0 0 0
- joint m_r3: origin xyz=0.5 2.25 1 rpy=0 0 0 -> xyz=0.5 1.5 1 rpy=0 0 0
