Commit message: evolve legs and length

File: bodies/body0.urdf (robot description, URDF)
Before this commit: robot robot, 5 links, 4 joints
Links:
- added link L1, mass 1; collision box size=1 0.2 0.2; visual box size=1 0.2 0.2
- added link LL1, mass 1; collision box size=0.2 0.2 1; visual box size=0.2 0.2 1
- added link r1, mass 1; collision box size=1 0.2 0.2; visual box size=1 0.2 0.2
- added link r2, mass 1; collision box size=1 0.2 0.2; visual box size=1 0.2 0.2
- added link rl1, mass 1; collision box size=0.2 0.2 1; visual box size=0.2 0.2 1
- added link rl2, mass 1; collision box size=0.2 0.2 1; visual box size=0.2 0.2 1
- link m: geometry collision box size=1 3 0.5; visual box size=1 3 0.5
Joints:
- added joint L1_LL1: type revolute, parent L1, child LL1, origin xyz=-1 0 0 rpy=0 0 0, axis 1 0 0, limit lower=-3.14159 upper=3.14159 effort=0.0 velocity=0.0
- added joint m_L1: type revolute, parent m, child L1, origin xyz=-0.5 0.5 1 rpy=0 0 0, axis 1 0 0, limit lower=-3.14159 upper=3.14159 effort=0.0 velocity=0.0
- added joint m_r1: type revolute, parent m, child r1, origin xyz=0.5 -0.16666666666666674 1 rpy=0 0 0, axis 1 0 0, limit lower=-3.14159 upper=3.14159 effort=0.0 velocity=0.0
- added joint m_r2: type revolute, parent m, child r2, origin xyz=0.5 1.1666666666666665 1 rpy=0 0 0, axis 1 0 0, limit lower=-3.14159 upper=3.14159 effort=0.0 velocity=0.0
- added joint r1_rl1: type revolute, parent r1, child rl1, origin xyz=1 0 0 rpy=0 0 0, axis 1 0 0, limit lower=-3.14159 upper=3.14159 effort=0.0 velocity=0.0
- added joint r2_rl2: type revolute, parent r2, child rl2, origin xyz=1 0 0 rpy=0 0 0, axis 1 0 0, limit lower=-3.14159 upper=3.14159 effort=0.0 velocity=0.0
- joint m_L0: origin xyz=-0.5 -3.0 1 rpy=0 0 0 -> xyz=-0.5 -1.5 1 rpy=0 0 0
- joint m_r0: origin xyz=0.5 -3.0 1 rpy=0 0 0 -> xyz=0.5 -1.5 1 rpy=0 0 0

File: bodies/body1.urdf (robot description, URDF)
Before this commit: robot robot, 5 links, 4 joints
Links:
- added link L1, mass 1; collision box size=1 0.2 0.2; visual box size=1 0.2 0.2
- added link LL1, mass 1; collision box size=0.2 0.2 1; visual box size=0.2 0.2 1
- added link r1, mass 1; collision box size=1 0.2 0.2; visual box size=1 0.2 0.2
- added link rl1, mass 1; collision box size=0.2 0.2 1; visual box size=0.2 0.2 1
- link m: geometry collision box size=1 5 0.5; visual box size=1 5 0.5
Joints:
- added joint L1_LL1: type revolute, parent L1, child LL1, origin xyz=-1 0 0 rpy=0 0 0, axis 1 0 0, limit lower=-3.14159 upper=3.14159 effort=0.0 velocity=0.0
- added joint m_L1: type revolute, parent m, child L1, origin xyz=-0.5 0.5 1 rpy=0 0 0, axis 1 0 0, limit lower=-3.14159 upper=3.14159 effort=0.0 velocity=0.0
- added joint m_r1: type revolute, parent m, child r1, origin xyz=0.5 0.5 1 rpy=0 0 0, axis 1 0 0, limit lower=-3.14159 upper=3.14159 effort=0.0 velocity=0.0
- added joint r1_rl1: type revolute, parent r1, child rl1, origin xyz=1 0 0 rpy=0 0 0, axis 1 0 0, limit lower=-3.14159 upper=3.14159 effort=0.0 velocity=0.0
- joint m_L0: origin xyz=-0.5 -3.0 1 rpy=0 0 0 -> xyz=-0.5 -2.5 1 rpy=0 0 0
- joint m_r0: origin xyz=0.5 -3.0 1 rpy=0 0 0 -> xyz=0.5 -2.5 1 rpy=0 0 0

File: bodies/body10.urdf (robot description, URDF)
Before this commit: robot robot, 9 links, 8 joints
Links:
- removed link r1
- removed link r2
- removed link rl1
- removed link rl2
- added link L1, mass 1; collision box size=1 0.2 0.2; visual box size=1 0.2 0.2
- added link L2, mass 1; collision box size=1 0.2 0.2; visual box size=1 0.2 0.2
- added link L3, mass 1; collision box size=1 0.2 0.2; visual box size=1 0.2 0.2
- added link LL1, mass 1; collision box size=0.2 0.2 1; visual box size=0.2 0.2 1
- added link LL2, mass 1; collision box size=0.2 0.2 1; visual box size=0.2 0.2 1
- added link LL3, mass 1; collision box size=0.2 0.2 1; visual box size=0.2 0.2 1
- link m: geometry collision box size=1 5 0.5; visual box size=1 5 0.5
Joints:
- removed joint m_r1
- removed joint m_r2
- removed joint r1_rl1
- removed joint r2_rl2
- added joint L1_LL1: type revolute, parent L1, child LL1, origin xyz=-1 0 0 rpy=0 0 0, axis 1 0 0, limit lower=-3.14159 upper=3.14159 effort=0.0 velocity=0.0
- added joint L2_LL2: type revolute, parent L2, child LL2, origin xyz=-1 0 0 rpy=0 0 0, axis 1 0 0, limit lower=-3.14159 upper=3.14159 effort=0.0 velocity=0.0
- added joint L3_LL3: type revolute, parent L3, child LL3, origin xyz=-1 0 0 rpy=0 0 0, axis 1 0 0, limit lower=-3.14159 upper=3.14159 effort=0.0 velocity=0.0
- added joint m_L1: type revolute, parent m, child L1, origin xyz=-0.5 -1.0 1 rpy=0 0 0, axis 1 0 0, limit lower=-3.14159 upper=3.14159 effort=0.0 velocity=0.0
- added joint m_L2: type revolute, parent m, child L2, origin xyz=-0.5 0.5 1 rpy=0 0 0, axis 1 0 0, limit lower=-3.14159 upper=3.14159 effort=0.0 velocity=0.0
- added joint m_L3: type revolute, parent m, child L3, origin xyz=-0.5 2.0 1 rpy=0 0 0, axis 1 0 0, limit lower=-3.14159 upper=3.14159 effort=0.0 velocity=0.0
- joint m_L0: origin xyz=-0.5 -3.5 1 rpy=0 0 0 -> xyz=-0.5 -2.5 1 rpy=0 0 0
- joint m_r0: origin xyz=0.5 -3.5 1 rpy=0 0 0 -> xyz=0.5 -2.5 1 rpy=0 0 0

File: bodies/body12.urdf (robot description, URDF)
Before this commit: robot robot, 7 links, 6 joints
Links:
- added link L1, mass 1; collision box size=1 0.2 0.2; visual box size=1 0.2 0.2
- added link L2, mass 1; collision box size=1 0.2 0.2; visual box size=1 0.2 0.2
- added link LL1, mass 1; collision box size=0.2 0.2 1; visual box size=0.2 0.2 1
- added link LL2, mass 1; collision box size=0.2 0.2 1; visual box size=0.2 0.2 1
- added link r2, mass 1; collision box size=1 0.2 0.2; visual box size=1 0.2 0.2
- added link r3, mass 1; collision box size=1 0.2 0.2; visual box size=1 0.2 0.2
- added link rl2, mass 1; collision box size=0.2 0.2 1; visual box size=0.2 0.2 1
- added link rl3, mass 1; collision box size=0.2 0.2 1; visual box size=0.2 0.2 1
- link m: geometry collision box size=1 3 0.5; visual box size=1 3 0.5
Joints:
- added joint L1_LL1: type revolute, parent L1, child LL1, origin xyz=-1 0 0 rpy=0 0 0, axis 1 0 0, limit lower=-3.14159 upper=3.14159 effort=0.0 velocity=0.0
- added joint L2_LL2: type revolute, parent L2, child LL2, origin xyz=-1 0 0 rpy=0 0 0, axis 1 0 0, limit lower=-3.14159 upper=3.14159 effort=0.0 velocity=0.0
- added joint m_L1: type revolute, parent m, child L1, origin xyz=-0.5 -0.16666666666666674 1 rpy=0 0 0, axis 1 0 0, limit lower=-3.14159 upper=3.14159 effort=0.0 velocity=0.0
- added joint m_L2: type revolute, parent m, child L2, origin xyz=-0.5 1.1666666666666665 1 rpy=0 0 0, axis 1 0 0, limit lower=-3.14159 upper=3.14159 effort=0.0 velocity=0.0
- added joint m_r2: type revolute, parent m, child r2, origin xyz=0.5 0.5 1 rpy=0 0 0, axis 1 0 0, limit lower=-3.14159 upper=3.14159 effort=0.0 velocity=0.0
- added joint m_r3: type revolute, parent m, child r3, origin xyz=0.5 1.5 1 rpy=0 0 0, axis 1 0 0, limit lower=-3.14159 upper=3.14159 effort=0.0 velocity=0.0
- added joint r2_rl2: type revolute, parent r2, child rl2, origin xyz=1 0 0 rpy=0 0 0, axis 1 0 0, limit lower=-3.14159 upper=3.14159 effort=0.0 velocity=0.0
- added joint r3_rl3: type revolute, parent r3, child rl3, origin xyz=1 0 0 rpy=0 0 0, axis 1 0 0, limit lower=-3.14159 upper=3.14159 effort=0.0 velocity=0.0
- joint m_L0: origin xyz=-0.5 -3.5 1 rpy=0 0 0 -> xyz=-0.5 -1.5 1 rpy=0 0 0
- joint m_r0: origin xyz=0.5 -3.5 1 rpy=0 0 0 -> xyz=0.5 -1.5 1 rpy=0 0 0
- joint m_r1: origin xyz=0.5 0.5 1 rpy=0 0 0 -> xyz=0.5 -0.5 1 rpy=0 0 0

File: bodies/body13.urdf (robot description, URDF)
Before this commit: robot robot, 9 links, 8 joints
Links:
- added link L1, mass 1; collision box size=1 0.2 0.2; visual box size=1 0.2 0.2
- added link L2, mass 1; collision box size=1 0.2 0.2; visual box size=1 0.2 0.2
- added link L3, mass 1; collision box size=1 0.2 0.2; visual box size=1 0.2 0.2
- added link LL1, mass 1; collision box size=0.2 0.2 1; visual box size=0.2 0.2 1
- added link LL2, mass 1; collision box size=0.2 0.2 1; visual box size=0.2 0.2 1
- added link LL3, mass 1; collision box size=0.2 0.2 1; visual box size=0.2 0.2 1
- link m: geometry collision box size=1 8 0.5; visual box size=1 8 0.5
Joints:
- added joint L1_LL1: type revolute, parent L1, child LL1, origin xyz=-1 0 0 rpy=0 0 0, axis 1 0 0, limit lower=-3.14159 upper=3.14159 effort=0.0 velocity=0.0
- added joint L2_LL2: type revolute, parent L2, child LL2, origin xyz=-1 0 0 rpy=0 0 0, axis 1 0 0, limit lower=-3.14159 upper=3.14159 effort=0.0 velocity=0.0
- added joint L3_LL3: type revolute, parent L3, child LL3, origin xyz=-1 0 0 rpy=0 0 0, axis 1 0 0, limit lower=-3.14159 upper=3.14159 effort=0.0 velocity=0.0
- added joint m_L1: type revolute, parent m, child L1, origin xyz=-0.5 -1.75 1 rpy=0 0 0, axis 1 0 0, limit lower=-3.14159 upper=3.14159 effort=0.0 velocity=0.0
- added joint m_L2: type revolute, parent m, child L2, origin xyz=-0.5 0.5 1 rpy=0 0 0, axis 1 0 0, limit lower=-3.14159 upper=3.14159 effort=0.0 velocity=0.0
- added joint m_L3: type revolute, parent m, child L3, origin xyz=-0.5 2.75 1 rpy=0 0 0, axis 1 0 0, limit lower=-3.14159 upper=3.14159 effort=0.0 velocity=0.0
- joint m_L0: origin xyz=-0.5 -2.5 1 rpy=0 0 0 -> xyz=-0.5 -4.0 1 rpy=0 0 0
- joint m_r0: origin xyz=0.5 -2.5 1 rpy=0 0 0 -> xyz=0.5 -4.0 1 rpy=0 0 0
- joint m_r1: origin xyz=0.5 -0.5 1 rpy=0 0 0 -> xyz=0.5 -1.0 1 rpy=0 0 0
- joint m_r2: origin xyz=0.5 1.5 1 rpy=0 0 0 -> xyz=0.5 2.0 1 rpy=0 0 0

File: bodies/body14.urdf (robot description, URDF)
Before this commit: robot robot, 13 links, 12 joints
Links:
- added link r2, mass 1; collision box size=1 0.2 0.2; visual box size=1 0.2 0.2
- added link rl2, mass 1; collision box size=0.2 0.2 1; visual box size=0.2 0.2 1
- link m: geometry collision box size=1 3 0.5; visual box size=1 3 0.5
Joints:
- added joint m_r2: type revolute, parent m, child r2, origin xyz=0.5 1.1666666666666665 1 rpy=0 0 0, axis 1 0 0, limit lower=-3.14159 upper=3.14159 effort=0.0 velocity=0.0
- added joint r2_rl2: type revolute, parent r2, child rl2, origin xyz=1 0 0 rpy=0 0 0, axis 1 0 0, limit lower=-3.14159 upper=3.14159 effort=0.0 velocity=0.0
- joint m_L0: origin xyz=-0.5 -3.5 1 rpy=0 0 0 -> xyz=-0.5 -1.5 1 rpy=0 0 0
- joint m_L1: origin xyz=-0.5 -1.5 1 rpy=0 0 0 -> xyz=-0.5 -0.5 1 rpy=0 0 0
- joint m_L3: origin xyz=-0.5 2.5 1 rpy=0 0 0 -> xyz=-0.5 1.5 1 rpy=0 0 0
- joint m_r0: origin xyz=0.5 -3.5 1 rpy=0 0 0 -> xyz=0.5 -1.5 1 rpy=0 0 0
- joint m_r1: origin xyz=0.5 0.5 1 rpy=0 0 0 -> xyz=0.5 -0.16666666666666674 1 rpy=0 0 0

File: bodies/body15.urdf (robot description, URDF)
Before this commit: robot robot, 11 links, 10 joints
Links:
- removed link r1
- removed link r2
- removed link r3
- removed link rl1
- removed link rl2
- removed link rl3
- added link L1, mass 1; collision box size=1 0.2 0.2; visual box size=1 0.2 0.2
- added link L2, mass 1; collision box size=1 0.2 0.2; visual box size=1 0.2 0.2
- added link L3, mass 1; collision box size=1 0.2 0.2; visual box size=1 0.2 0.2
- added link LL1, mass 1; collision box size=0.2 0.2 1; visual box size=0.2 0.2 1
- added link LL2, mass 1; collision box size=0.2 0.2 1; visual box size=0.2 0.2 1
- added link LL3, mass 1; collision box size=0.2 0.2 1; visual box size=0.2 0.2 1
- link m: geometry collision box size=1 8 0.5; visual box size=1 8 0.5
Joints:
- removed joint m_r1
- removed joint m_r2
- removed joint m_r3
- removed joint r1_rl1
- removed joint r2_rl2
- removed joint r3_rl3
- added joint L1_LL1: type revolute, parent L1, child LL1, origin xyz=-1 0 0 rpy=0 0 0, axis 1 0 0, limit lower=-3.14159 upper=3.14159 effort=0.0 velocity=0.0
- added joint L2_LL2: type revolute, parent L2, child LL2, origin xyz=-1 0 0 rpy=0 0 0, axis 1 0 0, limit lower=-3.14159 upper=3.14159 effort=0.0 velocity=0.0
- added joint L3_LL3: type revolute, parent L3, child LL3, origin xyz=-1 0 0 rpy=0 0 0, axis 1 0 0, limit lower=-3.14159 upper=3.14159 effort=0.0 velocity=0.0
- added joint m_L1: type revolute, parent m, child L1, origin xyz=-0.5 -1.75 1 rpy=0 0 0, axis 1 0 0, limit lower=-3.14159 upper=3.14159 effort=0.0 velocity=0.0
- added joint m_L2: type revolute, parent m, child L2, origin xyz=-0.5 0.5 1 rpy=0 0 0, axis 1 0 0, limit lower=-3.14159 upper=3.14159 effort=0.0 velocity=0.0
- added joint m_L3: type revolute, parent m, child L3, origin xyz=-0.5 2.75 1 rpy=0 0 0, axis 1 0 0, limit lower=-3.14159 upper=3.14159 effort=0.0 velocity=0.0
- joint m_L0: origin xyz=-0.5 -2.5 1 rpy=0 0 0 -> xyz=-0.5 -4.0 1 rpy=0 0 0
- joint m_r0: origin xyz=0.5 -2.5 1 rpy=0 0 0 -> xyz=0.5 -4.0 1 rpy=0 0 0

File: bodies/body16.urdf (robot description, URDF)
Before this commit: robot robot, 13 links, 12 joints
Links:
- removed link r1
- removed link rl1
- added link L4, mass 1; collision box size=1 0.2 0.2; visual box size=1 0.2 0.2
- added link LL4, mass 1; collision box size=0.2 0.2 1; visual box size=0.2 0.2 1
- link m: geometry collision box size=1 6 0.5; visual box size=1 6 0.5
Joints:
- removed joint m_r1
- removed joint r1_rl1
- added joint L4_LL4: type revolute, parent L4, child LL4, origin xyz=-1 0 0 rpy=0 0 0, axis 1 0 0, limit lower=-3.14159 upper=3.14159 effort=0.0 velocity=0.0
- added joint m_L4: type revolute, parent m, child L4, origin xyz=-0.5 2.5999999999999996 1 rpy=0 0 0, axis 1 0 0, limit lower=-3.14159 upper=3.14159 effort=0.0 velocity=0.0
- joint m_L0: origin xyz=-0.5 -2.0 1 rpy=0 0 0 -> xyz=-0.5 -3.0 1 rpy=0 0 0
- joint m_L1: origin xyz=-0.5 -0.75 1 rpy=0 0 0 -> xyz=-0.5 -1.6 1 rpy=0 0 0
- joint m_L2: origin xyz=-0.5 0.5 1 rpy=0 0 0 -> xyz=-0.5 -0.20000000000000018 1 rpy=0 0 0
- joint m_L3: origin xyz=-0.5 1.75 1 rpy=0 0 0 -> xyz=-0.5 1.1999999999999993 1 rpy=0 0 0
- joint m_r0: origin xyz=0.5 -2.0 1 rpy=0 0 0 -> xyz=0.5 -3.0 1 rpy=0 0 0

File: bodies/body17.urdf (robot description, URDF)
Before this commit: robot robot, 11 links, 10 joints
Links:
- added link r4, mass 1; collision box size=1 0.2 0.2; visual box size=1 0.2 0.2
- added link rl4, mass 1; collision box size=0.2 0.2 1; visual box size=0.2 0.2 1
- link m: geometry collision box size=1 7 0.5; visual box size=1 7 0.5
Joints:
- added joint m_r4: type revolute, parent m, child r4, origin xyz=0.5 2.9000000000000004 1 rpy=0 0 0, axis 1 0 0, limit lower=-3.14159 upper=3.14159 effort=0.0 velocity=0.0
- added joint r4_rl4: type revolute, parent r4, child rl4, origin xyz=1 0 0 rpy=0 0 0, axis 1 0 0, limit lower=-3.14159 upper=3.14159 effort=0.0 velocity=0.0
- joint m_L0: origin xyz=-0.5 -1.5 1 rpy=0 0 0 -> xyz=-0.5 -3.5 1 rpy=0 0 0
- joint m_r0: origin xyz=0.5 -1.5 1 rpy=0 0 0 -> xyz=0.5 -3.5 1 rpy=0 0 0
- joint m_r1: origin xyz=0.5 -0.5 1 rpy=0 0 0 -> xyz=0.5 -1.9 1 rpy=0 0 0
- joint m_r2: origin xyz=0.5 0.5 1 rpy=0 0 0 -> xyz=0.5 -0.2999999999999998 1 rpy=0 0 0
- joint m_r3: origin xyz=0.5 1.5 1 rpy=0 0 0 -> xyz=0.5 1.3000000000000007 1 rpy=0 0 0

File: bodies/body18.urdf (robot description, URDF)
Before this commit: robot robot, 17 links, 16 joints
Links:
- added link r3, mass 1; collision box size=1 0.2 0.2; visual box size=1 0.2 0.2
- added link rl3, mass 1; collision box size=0.2 0.2 1; visual box size=0.2 0.2 1
- link m: geometry collision box size=1 4 0.5; visual box size=1 4 0.5
Joints:
- added joint m_r3: type revolute, parent m, child r3, origin xyz=0.5 1.75 1 rpy=0 0 0, axis 1 0 0, limit lower=-3.14159 upper=3.14159 effort=0.0 velocity=0.0
- added joint r3_rl3: type revolute, parent r3, child rl3, origin xyz=1 0 0 rpy=0 0 0, axis 1 0 0, limit lower=-3.14159 upper=3.14159 effort=0.0 velocity=0.0
- joint m_L0: origin xyz=-0.5 -4.0 1 rpy=0 0 0 -> xyz=-0.5 -2.0 1 rpy=0 0 0
- joint m_L1: origin xyz=-0.5 -2.2 1 rpy=0 0 0 -> xyz=-0.5 -1.0 1 rpy=0 0 0
- joint m_L2: origin xyz=-0.5 -0.3999999999999999 1 rpy=0 0 0 -> xyz=-0.5 0.0 1 rpy=0 0 0
- joint m_L3: origin xyz=-0.5 1.4000000000000004 1 rpy=0 0 0 -> xyz=-0.5 1.0 1 rpy=0 0 0
- joint m_L4: origin xyz=-0.5 3.2 1 rpy=0 0 0 -> xyz=-0.5 2.0 1 rpy=0 0 0
- joint m_r0: origin xyz=0.5 -4.0 1 rpy=0 0 0 -> xyz=0.5 -2.0 1 rpy=0 0 0
- joint m_r1: origin xyz=0.5 -1.0 1 rpy=0 0 0 -> xyz=0.5 -0.75 1 rpy=0 0 0
- joint m_r2: origin xyz=0.5 2.0 1 rpy=0 0 0 -> xyz=0.5 0.5 1 rpy=0 0 0

File: bodies/body19.urdf (robot description, URDF)
Before this commit: robot robot, 17 links, 16 joints
Links:
- removed link L1
- removed link L2
- removed link LL1
- removed link LL2
- removed link r3
- removed link r4
- removed link rl3
- removed link rl4
- link m: geometry collision box size=1 5 0.5; visual box size=1 5 0.5
Joints:
- removed joint L1_LL1
- removed joint L2_LL2
- removed joint m_L1
- removed joint m_L2
- removed joint m_r3
- removed joint m_r4
- removed joint r3_rl3
- removed joint r4_rl4
- joint m_L0: origin xyz=-0.5 -3.0 1 rpy=0 0 0 -> xyz=-0.5 -2.5 1 rpy=0 0 0
- joint m_r0: origin xyz=0.5 -3.0 1 rpy=0 0 0 -> xyz=0.5 -2.5 1 rpy=0 0 0
- joint m_r1: origin xyz=0.5 -1.6 1 rpy=0 0 0 -> xyz=0.5 -0.5 1 rpy=0 0 0
- joint m_r2: origin xyz=0.5 -0.20000000000000018 1 rpy=0 0 0 -> xyz=0.5 1.5 1 rpy=0 0 0

File: bodies/body2.urdf (robot description, URDF)
Before this commit: robot robot, 5 links, 4 joints
Links:
- added link L1, mass 1; collision box size=1 0.2 0.2; visual box size=1 0.2 0.2
- added link L2, mass 1; collision box size=1 0.2 0.2; visual box size=1 0.2 0.2
- added link L3, mass 1; collision box size=1 0.2 0.2; visual box size=1 0.2 0.2
- added link L4, mass 1; collision box size=1 0.2 0.2; visual box size=1 0.2 0.2
- added link LL1, mass 1; collision box size=0.2 0.2 1; visual box size=0.2 0.2 1
- added link LL2, mass 1; collision box size=0.2 0.2 1; visual box size=0.2 0.2 1
- added link LL3, mass 1; collision box size=0.2 0.2 1; visual box size=0.2 0.2 1
- added link LL4, mass 1; collision box size=0.2 0.2 1; visual box size=0.2 0.2 1
- added link r1, mass 1; collision box size=1 0.2 0.2; visual box size=1 0.2 0.2
- added link r2, mass 1; collision box size=1 0.2 0.2; visual box size=1 0.2 0.2
- added link r3, mass 1; collision box size=1 0.2 0.2; visual box size=1 0.2 0.2
- added link r4, mass 1; collision box size=1 0.2 0.2; visual box size=1 0.2 0.2
- added link rl1, mass 1; collision box size=0.2 0.2 1; visual box size=0.2 0.2 1
- added link rl2, mass 1; collision box size=0.2 0.2 1; visual box size=0.2 0.2 1
- added link rl3, mass 1; collision box size=0.2 0.2 1; visual box size=0.2 0.2 1
- added link rl4, mass 1; collision box size=0.2 0.2 1; visual box size=0.2 0.2 1
- link m: geometry collision box size=1 8 0.5; visual box size=1 8 0.5
Joints:
- added joint L1_LL1: type revolute, parent L1, child LL1, origin xyz=-1 0 0 rpy=0 0 0, axis 1 0 0, limit lower=-3.14159 upper=3.14159 effort=0.0 velocity=0.0
- added joint L2_LL2: type revolute, parent L2, child LL2, origin xyz=-1 0 0 rpy=0 0 0, axis 1 0 0, limit lower=-3.14159 upper=3.14159 effort=0.0 velocity=0.0
- added joint L3_LL3: type revolute, parent L3, child LL3, origin xyz=-1 0 0 rpy=0 0 0, axis 1 0 0, limit lower=-3.14159 upper=3.14159 effort=0.0 velocity=0.0
- added joint L4_LL4: type revolute, parent L4, child LL4, origin xyz=-1 0 0 rpy=0 0 0, axis 1 0 0, limit lower=-3.14159 upper=3.14159 effort=0.0 velocity=0.0
- added joint m_L1: type revolute, parent m, child L1, origin xyz=-0.5 -2.2 1 rpy=0 0 0, axis 1 0 0, limit lower=-3.14159 upper=3.14159 effort=0.0 velocity=0.0
- added joint m_L2: type revolute, parent m, child L2, origin xyz=-0.5 -0.3999999999999999 1 rpy=0 0 0, axis 1 0 0, limit lower=-3.14159 upper=3.14159 effort=0.0 velocity=0.0
- added joint m_L3: type revolute, parent m, child L3, origin xyz=-0.5 1.4000000000000004 1 rpy=0 0 0, axis 1 0 0, limit lower=-3.14159 upper=3.14159 effort=0.0 velocity=0.0
- added joint m_L4: type revolute, parent m, child L4, origin xyz=-0.5 3.2 1 rpy=0 0 0, axis 1 0 0, limit lower=-3.14159 upper=3.14159 effort=0.0 velocity=0.0
- added joint m_r1: type revolute, parent m, child r1, origin xyz=0.5 -2.2 1 rpy=0 0 0, axis 1 0 0, limit lower=-3.14159 upper=3.14159 effort=0.0 velocity=0.0
- added joint m_r2: type revolute, parent m, child r2, origin xyz=0.5 -0.3999999999999999 1 rpy=0 0 0, axis 1 0 0, limit lower=-3.14159 upper=3.14159 effort=0.0 velocity=0.0
- added joint m_r3: type revolute, parent m, child r3, origin xyz=0.5 1.4000000000000004 1 rpy=0 0 0, axis 1 0 0, limit lower=-3.14159 upper=3.14159 effort=0.0 velocity=0.0
- added joint m_r4: type revolute, parent m, child r4, origin xyz=0.5 3.2 1 rpy=0 0 0, axis 1 0 0, limit lower=-3.14159 upper=3.14159 effort=0.0 velocity=0.0
- added joint r1_rl1: type revolute, parent r1, child rl1, origin xyz=1 0 0 rpy=0 0 0, axis 1 0 0, limit lower=-3.14159 upper=3.14159 effort=0.0 velocity=0.0
- added joint r2_rl2: type revolute, parent r2, child rl2, origin xyz=1 0 0 rpy=0 0 0, axis 1 0 0, limit lower=-3.14159 upper=3.14159 effort=0.0 velocity=0.0
- added joint r3_rl3: type revolute, parent r3, child rl3, origin xyz=1 0 0 rpy=0 0 0, axis 1 0 0, limit lower=-3.14159 upper=3.14159 effort=0.0 velocity=0.0
- added joint r4_rl4: type revolute, parent r4, child rl4, origin xyz=1 0 0 rpy=0 0 0, axis 1 0 0, limit lower=-3.14159 upper=3.14159 effort=0.0 velocity=0.0
- joint m_L0: origin xyz=-0.5 -3.0 1 rpy=0 0 0 -> xyz=-0.5 -4.0 1 rpy=0 0 0
- joint m_r0: origin xyz=0.5 -3.0 1 rpy=0 0 0 -> xyz=0.5 -4.0 1 rpy=0 0 0
