Commit message: evolve legs and length

File: bodies/body3.urdf (robot description, URDF)
Before this commit: robot robot, 5 links, 4 joints
Links:
- added link L1, mass 1; collision box size=1 0.2 0.2; visual box size=1 0.2 0.2
- added link L2, mass 1; collision box size=1 0.2 0.2; visual box size=1 0.2 0.2
- added link L3, mass 1; collision box size=1 0.2 0.2; visual box size=1 0.2 0.2
- added link L4, mass 1; collision box size=1 0.2 0.2; visual box size=1 0.2 0.2
- added link LL1, mass 1; collision box size=0.2 0.2 1; visual box size=0.2 0.2 1
- added link LL2, mass 1; collision box size=0.2 0.2 1; visual box size=0.2 0.2 1
- added link LL3, mass 1; collision box size=0.2 0.2 1; visual box size=0.2 0.2 1
- added link LL4, mass 1; collision box size=0.2 0.2 1; visual box size=0.2 0.2 1
- added link r1, mass 1; collision box size=1 0.2 0.2; visual box size=1 0.2 0.2
- added link rl1, mass 1; collision box size=0.2 0.2 1; visual box size=0.2 0.2 1
Joints:
- added joint L1_LL1: type revolute, parent L1, child LL1, origin xyz=-1 0 0 rpy=0 0 0, axis 1 0 0, limit lower=-3.14159 upper=3.14159 effort=0.0 velocity=0.0
- added joint L2_LL2: type revolute, parent L2, child LL2, origin xyz=-1 0 0 rpy=0 0 0, axis 1 0 0, limit lower=-3.14159 upper=3.14159 effort=0.0 velocity=0.0
- added joint L3_LL3: type revolute, parent L3, child LL3, origin xyz=-1 0 0 rpy=0 0 0, axis 1 0 0, limit lower=-3.14159 upper=3.14159 effort=0.0 velocity=0.0
- added joint L4_LL4: type revolute, parent L4, child LL4, origin xyz=-1 0 0 rpy=0 0 0, axis 1 0 0, limit lower=-3.14159 upper=3.14159 effort=0.0 velocity=0.0
- added joint m_L1: type revolute, parent m, child L1, origin xyz=-0.5 -1.6 1 rpy=0 0 0, axis 1 0 0, limit lower=-3.14159 upper=3.14159 effort=0.0 velocity=0.0
- added joint m_L2: type revolute, parent m, child L2, origin xyz=-0.5 -0.20000000000000018 1 rpy=0 0 0, axis 1 0 0, limit lower=-3.14159 upper=3.14159 effort=0.0 velocity=0.0
- added joint m_L3: type revolute, parent m, child L3, origin xyz=-0.5 1.1999999999999993 1 rpy=0 0 0, axis 1 0 0, limit lower=-3.14159 upper=3.14159 effort=0.0 velocity=0.0
- added joint m_L4: type revolute, parent m, child L4, origin xyz=-0.5 2.5999999999999996 1 rpy=0 0 0, axis 1 0 0, limit lower=-3.14159 upper=3.14159 effort=0.0 velocity=0.0
- added joint m_r1: type revolute, parent m, child r1, origin xyz=0.5 0.5 1 rpy=0 0 0, axis 1 0 0, limit lower=-3.14159 upper=3.14159 effort=0.0 velocity=0.0
- added joint r1_rl1: type revolute, parent r1, child rl1, origin xyz=1 0 0 rpy=0 0 0, axis 1 0 0, limit lower=-3.14159 upper=3.14159 effort=0.0 velocity=0.0

File: bodies/body4.urdf (robot description, URDF)
Before this commit: robot robot, 5 links, 4 joints
Links:
- added link L1, mass 1; collision box size=1 0.2 0.2; visual box size=1 0.2 0.2
- added link L2, mass 1; collision box size=1 0.2 0.2; visual box size=1 0.2 0.2
- added link L3, mass 1; collision box size=1 0.2 0.2; visual box size=1 0.2 0.2
- added link L4, mass 1; collision box size=1 0.2 0.2; visual box size=1 0.2 0.2
- added link LL1, mass 1; collision box size=0.2 0.2 1; visual box size=0.2 0.2 1
- added link LL2, mass 1; collision box size=0.2 0.2 1; visual box size=0.2 0.2 1
- added link LL3, mass 1; collision box size=0.2 0.2 1; visual box size=0.2 0.2 1
- added link LL4, mass 1; collision box size=0.2 0.2 1; visual box size=0.2 0.2 1
- added link r1, mass 1; collision box size=1 0.2 0.2; visual box size=1 0.2 0.2
- added link r2, mass 1; collision box size=1 0.2 0.2; visual box size=1 0.2 0.2
- added link r3, mass 1; collision box size=1 0.2 0.2; visual box size=1 0.2 0.2
- added link r4, mass 1; collision box size=1 0.2 0.2; visual box size=1 0.2 0.2
- added link rl1, mass 1; collision box size=0.2 0.2 1; visual box size=0.2 0.2 1
- added link rl2, mass 1; collision box size=0.2 0.2 1; visual box size=0.2 0.2 1
- added link rl3, mass 1; collision box size=0.2 0.2 1; visual box size=0.2 0.2 1
- added link rl4, mass 1; collision box size=0.2 0.2 1; visual box size=0.2 0.2 1
- link m: geometry collision box size=1 5 0.5; visual box size=1 5 0.5
Joints:
- added joint L1_LL1: type revolute, parent L1, child LL1, origin xyz=-1 0 0 rpy=0 0 0, axis 1 0 0, limit lower=-3.14159 upper=3.14159 effort=0.0 velocity=0.0
- added joint L2_LL2: type revolute, parent L2, child LL2, origin xyz=-1 0 0 rpy=0 0 0, axis 1 0 0, limit lower=-3.14159 upper=3.14159 effort=0.0 velocity=0.0
- added joint L3_LL3: type revolute, parent L3, child LL3, origin xyz=-1 0 0 rpy=0 0 0, axis 1 0 0, limit lower=-3.14159 upper=3.14159 effort=0.0 velocity=0.0
- added joint L4_LL4: type revolute, parent L4, child LL4, origin xyz=-1 0 0 rpy=0 0 0, axis 1 0 0, limit lower=-3.14159 upper=3.14159 effort=0.0 velocity=0.0
- added joint m_L1: type revolute, parent m, child L1, origin xyz=-0.5 -1.3 1 rpy=0 0 0, axis 1 0 0, limit lower=-3.14159 upper=3.14159 effort=0.0 velocity=0.0
- added joint m_L2: type revolute, parent m, child L2, origin xyz=-0.5 -0.10000000000000009 1 rpy=0 0 0, axis 1 0 0, limit lower=-3.14159 upper=3.14159 effort=0.0 velocity=0.0
- added joint m_L3: type revolute, parent m, child L3, origin xyz=-0.5 1.0999999999999996 1 rpy=0 0 0, axis 1 0 0, limit lower=-3.14159 upper=3.14159 effort=0.0 velocity=0.0
- added joint m_L4: type revolute, parent m, child L4, origin xyz=-0.5 2.3 1 rpy=0 0 0, axis 1 0 0, limit lower=-3.14159 upper=3.14159 effort=0.0 velocity=0.0
- added joint m_r1: type revolute, parent m, child r1, origin xyz=0.5 -1.3 1 rpy=0 0 0, axis 1 0 0, limit lower=-3.14159 upper=3.14159 effort=0.0 velocity=0.0
- added joint m_r2: type revolute, parent m, child r2, origin xyz=0.5 -0.10000000000000009 1 rpy=0 0 0, axis 1 0 0, limit lower=-3.14159 upper=3.14159 effort=0.0 velocity=0.0
- added joint m_r3: type revolute, parent m, child r3, origin xyz=0.5 1.0999999999999996 1 rpy=0 0 0, axis 1 0 0, limit lower=-3.14159 upper=3.14159 effort=0.0 velocity=0.0
- added joint m_r4: type revolute, parent m, child r4, origin xyz=0.5 2.3 1 rpy=0 0 0, axis 1 0 0, limit lower=-3.14159 upper=3.14159 effort=0.0 velocity=0.0
- added joint r1_rl1: type revolute, parent r1, child rl1, origin xyz=1 0 0 rpy=0 0 0, axis 1 0 0, limit lower=-3.14159 upper=3.14159 effort=0.0 velocity=0.0
- added joint r2_rl2: type revolute, parent r2, child rl2, origin xyz=1 0 0 rpy=0 0 0, axis 1 0 0, limit lower=-3.14159 upper=3.14159 effort=0.0 velocity=0.0
- added joint r3_rl3: type revolute, parent r3, child rl3, origin xyz=1 0 0 rpy=0 0 0, axis 1 0 0, limit lower=-3.14159 upper=3.14159 effort=0.0 velocity=0.0
- added joint r4_rl4: type revolute, parent r4, child rl4, origin xyz=1 0 0 rpy=0 0 0, axis 1 0 0, limit lower=-3.14159 upper=3.14159 effort=0.0 velocity=0.0
- joint m_L0: origin xyz=-0.5 -3.0 1 rpy=0 0 0 -> xyz=-0.5 -2.5 1 rpy=0 0 0
- joint m_r0: origin xyz=0.5 -3.0 1 rpy=0 0 0 -> xyz=0.5 -2.5 1 rpy=0 0 0

File: bodies/body6.urdf (robot description, URDF)
Before this commit: robot robot, 5 links, 4 joints
Links:
- added link L1, mass 1; collision box size=1 0.2 0.2; visual box size=1 0.2 0.2
- added link L2, mass 1; collision box size=1 0.2 0.2; visual box size=1 0.2 0.2
- added link L3, mass 1; collision box size=1 0.2 0.2; visual box size=1 0.2 0.2
- added link L4, mass 1; collision box size=1 0.2 0.2; visual box size=1 0.2 0.2
- added link LL1, mass 1; collision box size=0.2 0.2 1; visual box size=0.2 0.2 1
- added link LL2, mass 1; collision box size=0.2 0.2 1; visual box size=0.2 0.2 1
- added link LL3, mass 1; collision box size=0.2 0.2 1; visual box size=0.2 0.2 1
- added link LL4, mass 1; collision box size=0.2 0.2 1; visual box size=0.2 0.2 1
- added link r1, mass 1; collision box size=1 0.2 0.2; visual box size=1 0.2 0.2
- added link rl1, mass 1; collision box size=0.2 0.2 1; visual box size=0.2 0.2 1
- link m: geometry collision box size=1 5.5 0.5; visual box size=1 5.5 0.5
Joints:
- added joint L1_LL1: type revolute, parent L1, child LL1, origin xyz=-1 0 0 rpy=0 0 0, axis 1 0 0, limit lower=-3.14159 upper=3.14159 effort=0.0 velocity=0.0
- added joint L2_LL2: type revolute, parent L2, child LL2, origin xyz=-1 0 0 rpy=0 0 0, axis 1 0 0, limit lower=-3.14159 upper=3.14159 effort=0.0 velocity=0.0
- added joint L3_LL3: type revolute, parent L3, child LL3, origin xyz=-1 0 0 rpy=0 0 0, axis 1 0 0, limit lower=-3.14159 upper=3.14159 effort=0.0 velocity=0.0
- added joint L4_LL4: type revolute, parent L4, child LL4, origin xyz=-1 0 0 rpy=0 0 0, axis 1 0 0, limit lower=-3.14159 upper=3.14159 effort=0.0 velocity=0.0
- added joint m_L1: type revolute, parent m, child L1, origin xyz=-0.5 -1.45 1 rpy=0 0 0, axis 1 0 0, limit lower=-3.14159 upper=3.14159 effort=0.0 velocity=0.0
- added joint m_L2: type revolute, parent m, child L2, origin xyz=-0.5 -0.1499999999999999 1 rpy=0 0 0, axis 1 0 0, limit lower=-3.14159 upper=3.14159 effort=0.0 velocity=0.0
- added joint m_L3: type revolute, parent m, child L3, origin xyz=-0.5 1.1500000000000004 1 rpy=0 0 0, axis 1 0 0, limit lower=-3.14159 upper=3.14159 effort=0.0 velocity=0.0
- added joint m_L4: type revolute, parent m, child L4, origin xyz=-0.5 2.45 1 rpy=0 0 0, axis 1 0 0, limit lower=-3.14159 upper=3.14159 effort=0.0 velocity=0.0
- added joint m_r1: type revolute, parent m, child r1, origin xyz=0.5 0.5 1 rpy=0 0 0, axis 1 0 0, limit lower=-3.14159 upper=3.14159 effort=0.0 velocity=0.0
- added joint r1_rl1: type revolute, parent r1, child rl1, origin xyz=1 0 0 rpy=0 0 0, axis 1 0 0, limit lower=-3.14159 upper=3.14159 effort=0.0 velocity=0.0
- joint m_L0: origin xyz=-0.5 -3.0 1 rpy=0 0 0 -> xyz=-0.5 -2.75 1 rpy=0 0 0
- joint m_r0: origin xyz=0.5 -3.0 1 rpy=0 0 0 -> xyz=0.5 -2.75 1 rpy=0 0 0

File: bodies/body7.urdf (robot description, URDF)
Before this commit: robot robot, 5 links, 4 joints
Links:
- added link L1, mass 1; collision box size=1 0.2 0.2; visual box size=1 0.2 0.2
- added link L2, mass 1; collision box size=1 0.2 0.2; visual box size=1 0.2 0.2
- added link LL1, mass 1; collision box size=0.2 0.2 1; visual box size=0.2 0.2 1
- added link LL2, mass 1; collision box size=0.2 0.2 1; visual box size=0.2 0.2 1
- link m: geometry collision box size=1 7 0.5; visual box size=1 7 0.5
Joints:
- added joint L1_LL1: type revolute, parent L1, child LL1, origin xyz=-1 0 0 rpy=0 0 0, axis 1 0 0, limit lower=-3.14159 upper=3.14159 effort=0.0 velocity=0.0
- added joint L2_LL2: type revolute, parent L2, child LL2, origin xyz=-1 0 0 rpy=0 0 0, axis 1 0 0, limit lower=-3.14159 upper=3.14159 effort=0.0 velocity=0.0
- added joint m_L1: type revolute, parent m, child L1, origin xyz=-0.5 -0.8333333333333335 1 rpy=0 0 0, axis 1 0 0, limit lower=-3.14159 upper=3.14159 effort=0.0 velocity=0.0
- added joint m_L2: type revolute, parent m, child L2, origin xyz=-0.5 1.833333333333333 1 rpy=0 0 0, axis 1 0 0, limit lower=-3.14159 upper=3.14159 effort=0.0 velocity=0.0
- joint m_L0: origin xyz=-0.5 -3.0 1 rpy=0 0 0 -> xyz=-0.5 -3.5 1 rpy=0 0 0
- joint m_r0: origin xyz=0.5 -3.0 1 rpy=0 0 0 -> xyz=0.5 -3.5 1 rpy=0 0 0

File: bodies/body8.urdf (robot description, URDF)
Before this commit: robot robot, 5 links, 4 joints
Links:
- added link L1, mass 1; collision box size=1 0.2 0.2; visual box size=1 0.2 0.2
- added link L2, mass 1; collision box size=1 0.2 0.2; visual box size=1 0.2 0.2
- added link LL1, mass 1; collision box size=0.2 0.2 1; visual box size=0.2 0.2 1
- added link LL2, mass 1; collision box size=0.2 0.2 1; visual box size=0.2 0.2 1
- added link r1, mass 1; collision box size=1 0.2 0.2; visual box size=1 0.2 0.2
- added link r2, mass 1; collision box size=1 0.2 0.2; visual box size=1 0.2 0.2
- added link rl1, mass 1; collision box size=0.2 0.2 1; visual box size=0.2 0.2 1
- added link rl2, mass 1; collision box size=0.2 0.2 1; visual box size=0.2 0.2 1
Joints:
- added joint L1_LL1: type revolute, parent L1, child LL1, origin xyz=-1 0 0 rpy=0 0 0, axis 1 0 0, limit lower=-3.14159 upper=3.14159 effort=0.0 velocity=0.0
- added joint L2_LL2: type revolute, parent L2, child LL2, origin xyz=-1 0 0 rpy=0 0 0, axis 1 0 0, limit lower=-3.14159 upper=3.14159 effort=0.0 velocity=0.0
- added joint m_L1: type revolute, parent m, child L1, origin xyz=-0.5 -0.6666666666666665 1 rpy=0 0 0, axis 1 0 0, limit lower=-3.14159 upper=3.14159 effort=0.0 velocity=0.0
- added joint m_L2: type revolute, parent m, child L2, origin xyz=-0.5 1.666666666666667 1 rpy=0 0 0, axis 1 0 0, limit lower=-3.14159 upper=3.14159 effort=0.0 velocity=0.0
- added joint m_r1: type revolute, parent m, child r1, origin xyz=0.5 -0.6666666666666665 1 rpy=0 0 0, axis 1 0 0, limit lower=-3.14159 upper=3.14159 effort=0.0 velocity=0.0
- added joint m_r2: type revolute, parent m, child r2, origin xyz=0.5 1.666666666666667 1 rpy=0 0 0, axis 1 0 0, limit lower=-3.14159 upper=3.14159 effort=0.0 velocity=0.0
- added joint r1_rl1: type revolute, parent r1, child rl1, origin xyz=1 0 0 rpy=0 0 0, axis 1 0 0, limit lower=-3.14159 upper=3.14159 effort=0.0 velocity=0.0
- added joint r2_rl2: type revolute, parent r2, child rl2, origin xyz=1 0 0 rpy=0 0 0, axis 1 0 0, limit lower=-3.14159 upper=3.14159 effort=0.0 velocity=0.0

File: bodies/body9.urdf (robot description, URDF)
Before this commit: robot robot, 5 links, 4 joints
Links:
- added link L1, mass 1; collision box size=1 0.2 0.2; visual box size=1 0.2 0.2
- added link L2, mass 1; collision box size=1 0.2 0.2; visual box size=1 0.2 0.2
- added link LL1, mass 1; collision box size=0.2 0.2 1; visual box size=0.2 0.2 1
- added link LL2, mass 1; collision box size=0.2 0.2 1; visual box size=0.2 0.2 1
- added link r1, mass 1; collision box size=1 0.2 0.2; visual box size=1 0.2 0.2
- added link r2, mass 1; collision box size=1 0.2 0.2; visual box size=1 0.2 0.2
- added link r3, mass 1; collision box size=1 0.2 0.2; visual box size=1 0.2 0.2
- added link r4, mass 1; collision box size=1 0.2 0.2; visual box size=1 0.2 0.2
- added link rl1, mass 1; collision box size=0.2 0.2 1; visual box size=0.2 0.2 1
- added link rl2, mass 1; collision box size=0.2 0.2 1; visual box size=0.2 0.2 1
- added link rl3, mass 1; collision box size=0.2 0.2 1; visual box size=0.2 0.2 1
- added link rl4, mass 1; collision box size=0.2 0.2 1; visual box size=0.2 0.2 1
- link m: geometry collision box size=1 4 0.5; visual box size=1 4 0.5
Joints:
- added joint L1_LL1: type revolute, parent L1, child LL1, origin xyz=-1 0 0 rpy=0 0 0, axis 1 0 0, limit lower=-3.14159 upper=3.14159 effort=0.0 velocity=0.0
- added joint L2_LL2: type revolute, parent L2, child LL2, origin xyz=-1 0 0 rpy=0 0 0, axis 1 0 0, limit lower=-3.14159 upper=3.14159 effort=0.0 velocity=0.0
- added joint m_L1: type revolute, parent m, child L1, origin xyz=-0.5 -0.33333333333333326 1 rpy=0 0 0, axis 1 0 0, limit lower=-3.14159 upper=3.14159 effort=0.0 velocity=0.0
- added joint m_L2: type revolute, parent m, child L2, origin xyz=-0.5 1.3333333333333335 1 rpy=0 0 0, axis 1 0 0, limit lower=-3.14159 upper=3.14159 effort=0.0 velocity=0.0
- added joint m_r1: type revolute, parent m, child r1, origin xyz=0.5 -1.0 1 rpy=0 0 0, axis 1 0 0, limit lower=-3.14159 upper=3.14159 effort=0.0 velocity=0.0
- added joint m_r2: type revolute, parent m, child r2, origin xyz=0.5 0.0 1 rpy=0 0 0, axis 1 0 0, limit lower=-3.14159 upper=3.14159 effort=0.0 velocity=0.0
- added joint m_r3: type revolute, parent m, child r3, origin xyz=0.5 1.0 1 rpy=0 0 0, axis 1 0 0, limit lower=-3.14159 upper=3.14159 effort=0.0 velocity=0.0
- added joint m_r4: type revolute, parent m, child r4, origin xyz=0.5 2.0 1 rpy=0 0 0, axis 1 0 0, limit lower=-3.14159 upper=3.14159 effort=0.0 velocity=0.0
- added joint r1_rl1: type revolute, parent r1, child rl1, origin xyz=1 0 0 rpy=0 0 0, axis 1 0 0, limit lower=-3.14159 upper=3.14159 effort=0.0 velocity=0.0
- added joint r2_rl2: type revolute, parent r2, child rl2, origin xyz=1 0 0 rpy=0 0 0, axis 1 0 0, limit lower=-3.14159 upper=3.14159 effort=0.0 velocity=0.0
- added joint r3_rl3: type revolute, parent r3, child rl3, origin xyz=1 0 0 rpy=0 0 0, axis 1 0 0, limit lower=-3.14159 upper=3.14159 effort=0.0 velocity=0.0
- added joint r4_rl4: type revolute, parent r4, child rl4, origin xyz=1 0 0 rpy=0 0 0, axis 1 0 0, limit lower=-3.14159 upper=3.14159 effort=0.0 velocity=0.0
- joint m_L0: origin xyz=-0.5 -3.0 1 rpy=0 0 0 -> xyz=-0.5 -2.0 1 rpy=0 0 0
- joint m_r0: origin xyz=0.5 -3.0 1 rpy=0 0 0 -> xyz=0.5 -2.0 1 rpy=0 0 0

Commit message: generated body

File: bodies/body0.urdf (robot description, URDF)
Before this commit: robot robot, 11 links, 10 joints
Links:
- removed link LL0
- removed link LL1
- removed link m
- removed link r0
- removed link r1
- removed link r2
- removed link rl0
- removed link rl1
- removed link rl2
- added link L10, mass 1; collision box size=1.9136369871862604 1.539454680959811 1.391821395552055; visual box size=1.9136369871862604 1.539454680959811 1.391821395552055
- added link L11, mass 1; collision box size=1.8151640480039808 0.5746514157186347 1.2231187186401427; visual box size=1.8151640480039808 0.5746514157186347 1.2231187186401427
- added link L12, mass 1; collision box size=1.4202194106679682 1.8060776003435994 0.6391592422543633; visual box size=1.4202194106679682 1.8060776003435994 0.6391592422543633
- added link L13, mass 1; collision box size=0.345380385005746 0.5560435560489383 1.042222622220628; visual box size=0.345380385005746 0.5560435560489383 1.042222622220628
- added link L14, mass 1; collision box size=1.256568677020097 1.5330368974185777 0.721318820753057; visual box size=1.256568677020097 1.5330368974185777 0.721318820753057
- added link L15, mass 1; collision box size=0.6236270318291122 1.4462085225949142 0.46736165750563036; visual box size=0.6236270318291122 1.4462085225949142 0.46736165750563036
- added link L16, mass 1; collision box size=1.0944524443157952 0.27210285858762867 0.6252962796231698; visual box size=1.0944524443157952 0.27210285858762867 0.6252962796231698
- added link L17, mass 1; collision box size=2.147753227141714 0.584661441988658 0.8653955570500371; visual box size=2.147753227141714 0.584661441988658 0.8653955570500371
- added link L2, mass 1; collision box size=0.26377065312231324 0.985665550363817 0.3044675917571789; visual box size=0.26377065312231324 0.985665550363817 0.3044675917571789
- added link L3, mass 1; collision box size=1.5693742332146126 2.0277508853190445 1.0954109847533653; visual box size=1.5693742332146126 2.0277508853190445 1.0954109847533653
- added link L4, mass 1; collision box size=0.6247669905704594 0.7922986317606162 0.899090176483818; visual box size=0.6247669905704594 0.7922986317606162 0.899090176483818
- added link L5, mass 1; collision box size=1.576931430966888 0.31114364961015145 0.2798221040457614; visual box size=1.576931430966888 0.31114364961015145 0.2798221040457614
- added link L6, mass 1; collision box size=1.5413710797333564 1.8301875907257397 1.6063636734369722; visual box size=1.5413710797333564 1.8301875907257397 1.6063636734369722
- added link L7, mass 1; collision box size=1.6027327506703524 1.817106823126249 0.8630311757618321; visual box size=1.6027327506703524 1.817106823126249 0.8630311757618321
- added link L8, mass 1; collision box size=1.4931379170242467 1.299184464831802 0.5099498938249007; visual box size=1.4931379170242467 1.299184464831802 0.5099498938249007
- added link L9, mass 1; collision box size=1.0715450930915897 1.5003130281107167 1.148219382126143; visual box size=1.0715450930915897 1.5003130281107167 1.148219382126143
- link L0: geometry collision box size=1.0955229769305965 1.7977808854512831 0.7159394118864522; visual box size=1.0955229769305965 1.7977808854512831 0.7159394118864522
- link L1: geometry collision box size=1.8130690840706962 1.502807813606784 0.7573593046989755; visual box size=1.8130690840706962 1.502807813606784 0.7573593046989755
Joints:
- removed joint L0_LL0
- removed joint L1_LL1
- removed joint m_L0
- removed joint m_L1
- removed joint m_r0
- removed joint m_r1
- removed joint m_r2
- removed joint r0_rl0
- removed joint r1_rl1
- removed joint r2_rl2
- added joint L0_L1: type revolute, parent L0, child L1, origin xyz=0 0.8988904427256416 1 rpy=0 0 0, axis 1 0 0, limit lower=-3.14159 upper=3.14159 effort=0.0 velocity=0.0
- added joint L10_L11: type revolute, parent L10, child L11, origin xyz=0 1.539454680959811 0 rpy=0 0 0, axis 1 0 0, limit lower=-3.14159 upper=3.14159 effort=0.0 velocity=0.0
- added joint L11_L12: type revolute, parent L11, child L12, origin xyz=0 0.5746514157186347 0 rpy=0 0 0, axis 1 0 0, limit lower=-3.14159 upper=3.14159 effort=0.0 velocity=0.0
- added joint L12_L13: type revolute, parent L12, child L13, origin xyz=0 1.8060776003435994 0 rpy=0 0 0, axis 1 0 0, limit lower=-3.14159 upper=3.14159 effort=0.0 velocity=0.0
- added joint L13_L14: type revolute, parent L13, child L14, origin xyz=0 0.5560435560489383 0 rpy=0 0 0, axis 1 0 0, limit lower=-3.14159 upper=3.14159 effort=0.0 velocity=0.0
- added joint L14_L15: type revolute, parent L14, child L15, origin xyz=0 1.5330368974185777 0 rpy=0 0 0, axis 1 0 0, limit lower=-3.14159 upper=3.14159 effort=0.0 velocity=0.0
- added joint L15_L16: type revolute, parent L15, child L16, origin xyz=0 1.4462085225949142 0 rpy=0 0 0, axis 1 0 0, limit lower=-3.14159 upper=3.14159 effort=0.0 velocity=0.0
- added joint L16_L17: type revolute, parent L16, child L17, origin xyz=0 0.27210285858762867 0 rpy=0 0 0, axis 1 0 0, limit lower=-3.14159 upper=3.14159 effort=0.0 velocity=0.0
- added joint L1_L2: type revolute, parent L1, child L2, origin xyz=0 1.502807813606784 0 rpy=0 0 0, axis 1 0 0, limit lower=-3.14159 upper=3.14159 effort=0.0 velocity=0.0
- added joint L2_L3: type revolute, parent L2, child L3, origin xyz=0 0.985665550363817 0 rpy=0 0 0, axis 1 0 0, limit lower=-3.14159 upper=3.14159 effort=0.0 velocity=0.0
- added joint L3_L4: type revolute, parent L3, child L4, origin xyz=0 2.0277508853190445 0 rpy=0 0 0, axis 1 0 0, limit lower=-3.14159 upper=3.14159 effort=0.0 velocity=0.0
- added joint L4_L5: type revolute, parent L4, child L5, origin xyz=0 0.7922986317606162 0 rpy=0 0 0, axis 1 0 0, limit lower=-3.14159 upper=3.14159 effort=0.0 velocity=0.0
- added joint L5_L6: type revolute, parent L5, child L6, origin xyz=0 0.31114364961015145 0 rpy=0 0 0, axis 1 0 0, limit lower=-3.14159 upper=3.14159 effort=0.0 velocity=0.0
- added joint L6_L7: type revolute, parent L6, child L7, origin xyz=0 1.8301875907257397 0 rpy=0 0 0, axis 1 0 0, limit lower=-3.14159 upper=3.14159 effort=0.0 velocity=0.0
- added joint L7_L8: type revolute, parent L7, child L8, origin xyz=0 1.817106823126249 0 rpy=0 0 0, axis 1 0 0, limit lower=-3.14159 upper=3.14159 effort=0.0 velocity=0.0
- added joint L8_L9: type revolute, parent L8, child L9, origin xyz=0 1.299184464831802 0 rpy=0 0 0, axis 1 0 0, limit lower=-3.14159 upper=3.14159 effort=0.0 velocity=0.0
- added joint L9_L10: type revolute, parent L9, child L10, origin xyz=0 1.5003130281107167 0 rpy=0 0 0, axis 1 0 0, limit lower=-3.14159 upper=3.14159 effort=0.0 velocity=0.0
