Commit message: a6

File: bodies/body0.urdf (robot description, URDF)
Before this commit: robot robot, 18 links, 17 joints
Links:
- removed link L16
- removed link L17
- link L0: geometry collision box size=1.9408820300041787 0.6738647669347573 0.6314064191164128; visual box size=1.9408820300041787 0.6738647669347573 0.6314064191164128
- link L1: geometry collision box size=1.6157115798213557 1.2129627689722018 1.4025950710457114; visual box size=1.6157115798213557 1.2129627689722018 1.4025950710457114
- link L10: geometry collision box size=1.4806367331618928 1.7896186699956602 0.28630218601808416; visual box size=1.4806367331618928 1.7896186699956602 0.28630218601808416
- link L11: geometry collision box size=0.7360819072035074 1.5475896253322312 0.7310160839971527; visual box size=0.7360819072035074 1.5475896253322312 0.7310160839971527
- link L12: geometry collision box size=0.5791906553823869 1.3260773958381693 2.0622488692292107; visual box size=0.5791906553823869 1.3260773958381693 2.0622488692292107
- link L13: geometry collision box size=0.8349176789212471 0.7667986074800694 1.94065668530528; visual box size=0.8349176789212471 0.7667986074800694 1.94065668530528
- link L14: geometry collision box size=0.42629822147685986 1.7867211110342989 1.6542036257369541; visual box size=0.42629822147685986 1.7867211110342989 1.6542036257369541
- link L15: geometry collision box size=1.0708220369124961 1.7424924076194397 1.276072496939377; visual box size=1.0708220369124961 1.7424924076194397 1.276072496939377
- link L2: geometry collision box size=1.0121781614799192 0.5783200983028225 1.7882913267680458; visual box size=1.0121781614799192 0.5783200983028225 1.7882913267680458
- link L3: geometry collision box size=0.4100938124312908 0.6439212070858891 0.4914770454212772; visual box size=0.4100938124312908 0.6439212070858891 0.4914770454212772
- link L4: geometry collision box size=1.821422760098992 1.7739908260934643 1.4317832035868914; visual box size=1.821422760098992 1.7739908260934643 1.4317832035868914
- link L5: geometry collision box size=0.6029186477934889 1.8212526239444269 0.21952505057431876; visual box size=0.6029186477934889 1.8212526239444269 0.21952505057431876
- link L6: geometry collision box size=1.4180384878639747 1.5065506635460149 1.0167945247656416; visual box size=1.4180384878639747 1.5065506635460149 1.0167945247656416
- link L7: geometry collision box size=0.516396462246395 0.21593074334711498 0.6963608639018048; visual box size=0.516396462246395 0.21593074334711498 0.6963608639018048
- link L8: geometry collision box size=2.1033154898510196 1.4754228366874247 0.9423601102563097; visual box size=2.1033154898510196 1.4754228366874247 0.9423601102563097
- link L9: geometry collision box size=1.2126764457905985 0.6191574932504531 2.1793957611723638; visual box size=1.2126764457905985 0.6191574932504531 2.1793957611723638
Joints:
- removed joint L15_L16
- removed joint L16_L17
- joint L0_L1: origin xyz=0 0.8988904427256416 1 rpy=0 0 0 -> xyz=0 0.33693238346737864 1 rpy=0 0 0
- joint L10_L11: axis 1 0 0 -> 1 1 0; origin xyz=0 1.539454680959811 0 rpy=0 0 0 -> xyz=0 1.7896186699956602 0 rpy=0 0 0
- joint L11_L12: axis 1 0 0 -> 1 1 0; origin xyz=0 0.5746514157186347 0 rpy=0 0 0 -> xyz=0 1.5475896253322312 0 rpy=0 0 0
- joint L12_L13: axis 1 0 0 -> 1 1 0; origin xyz=0 1.8060776003435994 0 rpy=0 0 0 -> xyz=0 1.3260773958381693 0 rpy=0 0 0
- joint L13_L14: axis 1 0 0 -> 1 1 0; origin xyz=0 0.5560435560489383 0 rpy=0 0 0 -> xyz=0 0.7667986074800694 0 rpy=0 0 0
- joint L14_L15: axis 1 0 0 -> 1 1 0; origin xyz=0 1.5330368974185777 0 rpy=0 0 0 -> xyz=0 1.7867211110342989 0 rpy=0 0 0
- joint L1_L2: axis 1 0 0 -> 1 1 0; origin xyz=0 1.502807813606784 0 rpy=0 0 0 -> xyz=0 1.2129627689722018 0 rpy=0 0 0
- joint L2_L3: axis 1 0 0 -> 1 1 0; origin xyz=0 0.985665550363817 0 rpy=0 0 0 -> xyz=0 0.5783200983028225 0 rpy=0 0 0
- joint L3_L4: axis 1 0 0 -> 1 1 0; origin xyz=0 2.0277508853190445 0 rpy=0 0 0 -> xyz=0 0.6439212070858891 0 rpy=0 0 0
- joint L4_L5: axis 1 0 0 -> 1 1 0; origin xyz=0 0.7922986317606162 0 rpy=0 0 0 -> xyz=0 1.7739908260934643 0 rpy=0 0 0
- joint L5_L6: axis 1 0 0 -> 1 1 0; origin xyz=0 0.31114364961015145 0 rpy=0 0 0 -> xyz=0 1.8212526239444269 0 rpy=0 0 0
- joint L6_L7: axis 1 0 0 -> 1 1 0; origin xyz=0 1.8301875907257397 0 rpy=0 0 0 -> xyz=0 1.5065506635460149 0 rpy=0 0 0
- joint L7_L8: axis 1 0 0 -> 1 1 0; origin xyz=0 1.817106823126249 0 rpy=0 0 0 -> xyz=0 0.21593074334711498 0 rpy=0 0 0
- joint L8_L9: axis 1 0 0 -> 1 1 0; origin xyz=0 1.299184464831802 0 rpy=0 0 0 -> xyz=0 1.4754228366874247 0 rpy=0 0 0
- joint L9_L10: axis 1 0 0 -> 1 1 0; origin xyz=0 1.5003130281107167 0 rpy=0 0 0 -> xyz=0 0.6191574932504531 0 rpy=0 0 0

Commit message: started

File: bodies/body0.urdf (robot description, URDF)
Before this commit: robot robot, 16 links, 15 joints
Links:
- added link L16, mass 1; collision box size=0.30301974652354274 0.52644404194894 0.9529420043628458; visual box size=0.30301974652354274 0.52644404194894 0.9529420043628458
- added link L17, mass 1; collision box size=1.6113141324520046 1.1483708722168946 0.3479205857531383; visual box size=1.6113141324520046 1.1483708722168946 0.3479205857531383
- added link L18, mass 1; collision box size=1.0632952582157422 0.8111386898710622 1.5294200638873072; visual box size=1.0632952582157422 0.8111386898710622 1.5294200638873072
- added link L19, mass 1; collision box size=2.041836332369775 0.29607605541799625 1.1110878068765726; visual box size=2.041836332369775 0.29607605541799625 1.1110878068765726
- added link L20, mass 1; collision box size=2.054949027915298 1.8422514733486854 1.633402227925164; visual box size=2.054949027915298 1.8422514733486854 1.633402227925164
- added link L21, mass 1; collision box size=0.4359234594586477 0.8293824491978923 0.7812172694556925; visual box size=0.4359234594586477 0.8293824491978923 0.7812172694556925
- added link L22, mass 1; collision box size=0.21869021332020117 1.8643651679005397 1.0854884952492614; visual box size=0.21869021332020117 1.8643651679005397 1.0854884952492614
- added link L23, mass 1; collision box size=2.0662523438037836 1.061101093914441 1.4085599411221397; visual box size=2.0662523438037836 1.061101093914441 1.4085599411221397
- added link L24, mass 1; collision box size=0.6420461011808414 1.1505782296902596 0.947774117619868; visual box size=0.6420461011808414 1.1505782296902596 0.947774117619868
- link L0: geometry collision box size=0.5215612052703498 0.6131110337814754 1.3650745494647145; visual box size=0.5215612052703498 0.6131110337814754 1.3650745494647145
- link L1: geometry collision box size=1.8317573973917272 2.0195402589257774 0.7678073669735697; visual box size=1.8317573973917272 2.0195402589257774 0.7678073669735697
- link L10: geometry collision box size=1.0518740200295447 0.21592207127016178 1.567868851223533; visual box size=1.0518740200295447 0.21592207127016178 1.567868851223533
- link L11: geometry collision box size=1.563242280591874 0.6049312110666929 0.36271626743692026; visual box size=1.563242280591874 0.6049312110666929 0.36271626743692026
- link L12: geometry collision box size=1.088020355962649 0.9201554964510403 0.3854041769796986; visual box size=1.088020355962649 0.9201554964510403 0.3854041769796986
- link L13: geometry collision box size=1.2249215413280936 2.0933607720142784 2.1212794221084397; visual box size=1.2249215413280936 2.0933607720142784 2.1212794221084397
- link L14: geometry collision box size=2.0370105747993192 0.6828756403409926 0.2175189910514415; visual box size=2.0370105747993192 0.6828756403409926 0.2175189910514415
- link L15: geometry collision box size=1.3692871980916432 1.5722507289100984 1.1124941164570128; visual box size=1.3692871980916432 1.5722507289100984 1.1124941164570128
- link L2: geometry collision box size=0.905917589038338 1.0768457239265052 0.5745952023068568; visual box size=0.905917589038338 1.0768457239265052 0.5745952023068568
- link L3: geometry collision box size=0.9865226275534944 1.6696190993651272 1.2138223945758577; visual box size=0.9865226275534944 1.6696190993651272 1.2138223945758577
- link L4: geometry collision box size=0.9591194400448184 1.73974667233193 1.543562500266677; visual box size=0.9591194400448184 1.73974667233193 1.543562500266677
- link L5: geometry collision box size=2.104337669180767 0.2961387539289316 1.5407938525680411; visual box size=2.104337669180767 0.2961387539289316 1.5407938525680411
- link L6: geometry collision box size=2.062839092440494 0.3445278794197802 0.9823134717110826; visual box size=2.062839092440494 0.3445278794197802 0.9823134717110826
- link L7: geometry collision box size=2.023308844568038 0.9642748043084299 2.0792761174743126; visual box size=2.023308844568038 0.9642748043084299 2.0792761174743126
- link L8: geometry collision box size=0.5012674079997508 0.7916349984392397 0.45072929913342535; visual box size=0.5012674079997508 0.7916349984392397 0.45072929913342535
- link L9: geometry collision box size=0.7095380088374506 1.2744701357201589 0.9644227090350461; visual box size=0.7095380088374506 1.2744701357201589 0.9644227090350461
Joints:
- added joint L15_L16: type revolute, parent L15, child L16, origin xyz=0 1.5722507289100984 0 rpy=0 0 0, axis 1 1 0, limit lower=-3.14159 upper=3.14159 effort=0.0 velocity=0.0
- added joint L16_L17: type revolute, parent L16, child L17, origin xyz=0 0.52644404194894 0 rpy=0 0 0, axis 1 1 0, limit lower=-3.14159 upper=3.14159 effort=0.0 velocity=0.0
- added joint L17_L18: type revolute, parent L17, child L18, origin xyz=0 1.1483708722168946 0 rpy=0 0 0, axis 1 1 0, limit lower=-3.14159 upper=3.14159 effort=0.0 velocity=0.0
- added joint L18_L19: type revolute, parent L18, child L19, origin xyz=0 0.8111386898710622 0 rpy=0 0 0, axis 1 1 0, limit lower=-3.14159 upper=3.14159 effort=0.0 velocity=0.0
- added joint L19_L20: type revolute, parent L19, child L20, origin xyz=0 0.29607605541799625 0 rpy=0 0 0, axis 1 1 0, limit lower=-3.14159 upper=3.14159 effort=0.0 velocity=0.0
- added joint L20_L21: type revolute, parent L20, child L21, origin xyz=0 1.8422514733486854 0 rpy=0 0 0, axis 1 1 0, limit lower=-3.14159 upper=3.14159 effort=0.0 velocity=0.0
- added joint L21_L22: type revolute, parent L21, child L22, origin xyz=0 0.8293824491978923 0 rpy=0 0 0, axis 1 1 0, limit lower=-3.14159 upper=3.14159 effort=0.0 velocity=0.0
- added joint L22_L23: type revolute, parent L22, child L23, origin xyz=0 1.8643651679005397 0 rpy=0 0 0, axis 1 1 0, limit lower=-3.14159 upper=3.14159 effort=0.0 velocity=0.0
- added joint L23_L24: type revolute, parent L23, child L24, origin xyz=0 1.061101093914441 0 rpy=0 0 0, axis 1 1 0, limit lower=-3.14159 upper=3.14159 effort=0.0 velocity=0.0
- joint L0_L1: origin xyz=0 0.33693238346737864 1 rpy=0 0 0 -> xyz=0 0.3065555168907377 1 rpy=0 0 0
- joint L10_L11: origin xyz=0 1.7896186699956602 0 rpy=0 0 0 -> xyz=0 0.21592207127016178 0 rpy=0 0 0
- joint L11_L12: origin xyz=0 1.5475896253322312 0 rpy=0 0 0 -> xyz=0 0.6049312110666929 0 rpy=0 0 0
- joint L12_L13: origin xyz=0 1.3260773958381693 0 rpy=0 0 0 -> xyz=0 0.9201554964510403 0 rpy=0 0 0
- joint L13_L14: origin xyz=0 0.7667986074800694 0 rpy=0 0 0 -> xyz=0 2.0933607720142784 0 rpy=0 0 0
- joint L14_L15: origin xyz=0 1.7867211110342989 0 rpy=0 0 0 -> xyz=0 0.6828756403409926 0 rpy=0 0 0
- joint L1_L2: origin xyz=0 1.2129627689722018 0 rpy=0 0 0 -> xyz=0 2.0195402589257774 0 rpy=0 0 0
- joint L2_L3: origin xyz=0 0.5783200983028225 0 rpy=0 0 0 -> xyz=0 1.0768457239265052 0 rpy=0 0 0
- joint L3_L4: origin xyz=0 0.6439212070858891 0 rpy=0 0 0 -> xyz=0 1.6696190993651272 0 rpy=0 0 0
- joint L4_L5: origin xyz=0 1.7739908260934643 0 rpy=0 0 0 -> xyz=0 1.73974667233193 0 rpy=0 0 0
- joint L5_L6: origin xyz=0 1.8212526239444269 0 rpy=0 0 0 -> xyz=0 0.2961387539289316 0 rpy=0 0 0
- joint L6_L7: origin xyz=0 1.5065506635460149 0 rpy=0 0 0 -> xyz=0 0.3445278794197802 0 rpy=0 0 0
- joint L7_L8: origin xyz=0 0.21593074334711498 0 rpy=0 0 0 -> xyz=0 0.9642748043084299 0 rpy=0 0 0
- joint L8_L9: origin xyz=0 1.4754228366874247 0 rpy=0 0 0 -> xyz=0 0.7916349984392397 0 rpy=0 0 0
- joint L9_L10: origin xyz=0 0.6191574932504531 0 rpy=0 0 0 -> xyz=0 1.2744701357201589 0 rpy=0 0 0

Commit message: working without sensors or motors

File: bodies/body0.urdf (robot description, URDF)
Before this commit: robot robot, 25 links, 24 joints
Links:
- removed link L0
- removed link L1
- removed link L10
- removed link L11
- removed link L12
- removed link L13
- removed link L14
- removed link L15
- removed link L16
- removed link L17
- removed link L18
- removed link L19
- removed link L2
- removed link L20
- removed link L21
- removed link L22
- removed link L23
- removed link L24
- removed link L3
- removed link L4
- removed link L5
- removed link L6
- removed link L7
- removed link L8
- removed link L9
- added link rootLink, mass 1; collision box size=1 1 1; visual box size=1 1 1
- added link rootLink0, mass 1; collision box size=1 1.6270003965398545 1; visual box size=1 1.6270003965398545 1
- added link rootLink00, mass 1; collision box size=1 1 1.5872028841260102; visual box size=1 1 1.5872028841260102
- added link rootLink000, mass 1; collision box size=1 1 1.4005991779394051; visual box size=1 1 1.4005991779394051
- added link rootLink001, mass 1; collision box size=1.1866318579054815 1 1; visual box size=1.1866318579054815 1 1
- added link rootLink003, mass 1; collision box size=1 1.1901944018261443 1; visual box size=1 1.1901944018261443 1
- added link rootLink0030, mass 1; collision box size=1 1 1.9610610910638906; visual box size=1 1 1.9610610910638906
- added link rootLink00300, mass 1; collision box size=1 1 1.0036196015222512; visual box size=1 1 1.0036196015222512
- added link rootLink00301, mass 1; collision box size=1.082534144799488 1 1; visual box size=1.082534144799488 1 1
- added link rootLink00304, mass 1; collision box size=1 1.7691068602628972 1; visual box size=1 1.7691068602628972 1
- added link rootLink0031, mass 1; collision box size=1 1.8664802929115392 1; visual box size=1 1.8664802929115392 1
- added link rootLink00310, mass 1; collision box size=1 1.2465819165906464 1; visual box size=1 1.2465819165906464 1
- added link rootLink00311, mass 1; collision box size=1.6939134788058037 1 1; visual box size=1.6939134788058037 1 1
- added link rootLink01, mass 1; collision box size=1.8479591261103465 1 1; visual box size=1.8479591261103465 1 1
- added link rootLink010, mass 1; collision box size=1 1 1.5945449284466064; visual box size=1 1 1.5945449284466064
- added link rootLink011, mass 1; collision box size=1.2239351085776338 1 1; visual box size=1.2239351085776338 1 1
- added link rootLink03, mass 1; collision box size=1 1.870881871060347 1; visual box size=1 1.870881871060347 1
Joints:
- removed joint L0_L1
- removed joint L10_L11
- removed joint L11_L12
- removed joint L12_L13
- removed joint L13_L14
- removed joint L14_L15
- removed joint L15_L16
- removed joint L16_L17
- removed joint L17_L18
- removed joint L18_L19
- removed joint L19_L20
- removed joint L1_L2
- removed joint L20_L21
- removed joint L21_L22
- removed joint L22_L23
- removed joint L23_L24
- removed joint L2_L3
- removed joint L3_L4
- removed joint L4_L5
- removed joint L5_L6
- removed joint L6_L7
- removed joint L7_L8
- removed joint L8_L9
- removed joint L9_L10
- added joint rootLink0030_rootLink00300: type revolute, parent rootLink0030, child rootLink00300, origin xyz=0 0 1.9610610910638906 rpy=0 0 0, axis 0 1 0, limit lower=-3.14159 upper=3.14159 effort=0.0 velocity=0.0
- added joint rootLink0030_rootLink00301: type revolute, parent rootLink0030, child rootLink00301, origin xyz=0.5 0 0.9805305455319453 rpy=0 0 0, axis 1 0 0, limit lower=-3.14159 upper=3.14159 effort=0.0 velocity=0.0
- added joint rootLink0030_rootLink00304: type revolute, parent rootLink0030, child rootLink00304, origin xyz=0 0.5 0.9805305455319453 rpy=0 0 0, axis 0 0 1, limit lower=-3.14159 upper=3.14159 effort=0.0 velocity=0.0
- added joint rootLink0031_rootLink00310: type revolute, parent rootLink0031, child rootLink00310, origin xyz=0 1.8664802929115392 0 rpy=0 0 0, axis 0 1 0, limit lower=-3.14159 upper=3.14159 effort=0.0 velocity=0.0
- added joint rootLink0031_rootLink00311: type revolute, parent rootLink0031, child rootLink00311, origin xyz=0.5 0.9332401464557696 0 rpy=0 0 0, axis 0 0 1, limit lower=-3.14159 upper=3.14159 effort=0.0 velocity=0.0
- added joint rootLink003_rootLink0030: type revolute, parent rootLink003, child rootLink0030, origin xyz=0 0.5950972009130722 0.5 rpy=0 0 0, axis 0 0 1, limit lower=-3.14159 upper=3.14159 effort=0.0 velocity=0.0
- added joint rootLink003_rootLink0031: type revolute, parent rootLink003, child rootLink0031, origin xyz=0 1.1901944018261443 0 rpy=0 0 0, axis 0 0 1, limit lower=-3.14159 upper=3.14159 effort=0.0 velocity=0.0
- added joint rootLink00_rootLink000: type revolute, parent rootLink00, child rootLink000, origin xyz=0 0 1.5872028841260102 rpy=0 0 0, axis 0 1 0, limit lower=-3.14159 upper=3.14159 effort=0.0 velocity=0.0
- added joint rootLink00_rootLink001: type revolute, parent rootLink00, child rootLink001, origin xyz=0.5 0 0.7936014420630051 rpy=0 0 0, axis 0 0 1, limit lower=-3.14159 upper=3.14159 effort=0.0 velocity=0.0
- added joint rootLink00_rootLink003: type revolute, parent rootLink00, child rootLink003, origin xyz=0 0.5 0.7936014420630051 rpy=0 0 0, axis 0 0 1, limit lower=-3.14159 upper=3.14159 effort=0.0 velocity=0.0
- added joint rootLink01_rootLink010: type revolute, parent rootLink01, child rootLink010, origin xyz=0.9239795630551733 0 0.5 rpy=0 0 0, axis 0 0 1, limit lower=-3.14159 upper=3.14159 effort=0.0 velocity=0.0
- added joint rootLink01_rootLink011: type revolute, parent rootLink01, child rootLink011, origin xyz=1.8479591261103465 0 0 rpy=0 0 0, axis 0 0 1, limit lower=-3.14159 upper=3.14159 effort=0.0 velocity=0.0
- added joint rootLink0_rootLink00: type revolute, parent rootLink0, child rootLink00, origin xyz=0 0.8135001982699273 0.5 rpy=0 0 0, axis 0 1 0, limit lower=-3.14159 upper=3.14159 effort=0.0 velocity=0.0
- added joint rootLink0_rootLink01: type revolute, parent rootLink0, child rootLink01, origin xyz=0.5 0.8135001982699273 0 rpy=0 0 0, axis 0 0 1, limit lower=-3.14159 upper=3.14159 effort=0.0 velocity=0.0
- added joint rootLink0_rootLink03: type revolute, parent rootLink0, child rootLink03, origin xyz=0 1.6270003965398545 0 rpy=0 0 0, axis 1 0 0, limit lower=-3.14159 upper=3.14159 effort=0.0 velocity=0.0
- added joint rootLink_rootLink0: type revolute, parent rootLink, child rootLink0, origin xyz=0 0.5 0.5 rpy=0 0 0, axis 1 0 0, limit lower=-3.14159 upper=3.14159 effort=0.0 velocity=0.0
