Commit message: finished assgnment 7

File: bodies/body0.urdf (robot description, URDF)
Before this commit: robot robot, 17 links, 16 joints
Links:
- removed link rootLink003
- removed link rootLink0030
- removed link rootLink00300
- removed link rootLink00301
- removed link rootLink00304
- removed link rootLink0031
- removed link rootLink00310
- removed link rootLink00311
- removed link rootLink010
- removed link rootLink011
- added link rootLink0000, mass 1; collision box size=1 1.045989620724986 1; visual box size=1 1.045989620724986 1
- added link rootLink0010, mass 1; collision box size=1 1 1.802701461242789; visual box size=1 1 1.802701461242789
- added link rootLink00100, mass 1; collision box size=1 1 1.8397949731803716; visual box size=1 1 1.8397949731803716
- added link rootLink00101, mass 1; collision box size=1 1.0772987139357206 1; visual box size=1 1.0772987139357206 1
- added link rootLink030, mass 1; collision box size=1.0327212158238008 1 1; visual box size=1.0327212158238008 1 1
- added link rootLink1, mass 1; collision box size=1 1 1.982059288687386; visual box size=1 1 1.982059288687386
- added link rootLink10, mass 1; collision box size=1.8882580595076672 1 1; visual box size=1.8882580595076672 1 1
- added link rootLink100, mass 1; collision box size=1 1.0813387183155512 1; visual box size=1 1.0813387183155512 1
- added link rootLink1000, mass 1; collision box size=1 1.5486971344555105 1; visual box size=1 1.5486971344555105 1
- added link rootLink1002, mass 1; collision box size=1.0910125194246736 1 1; visual box size=1.0910125194246736 1 1
- added link rootLink10020, mass 1; collision box size=1.1588896168180487 1 1; visual box size=1.1588896168180487 1 1
- added link rootLink10022, mass 1; collision box size=1 1.3023813282603252 1; visual box size=1 1.3023813282603252 1
- added link rootLink12, mass 1; collision box size=1 1 1.618469756887444; visual box size=1 1 1.618469756887444
- link rootLink0: geometry collision box size=1 1.7404012319607065 1; visual box size=1 1.7404012319607065 1
- link rootLink00: geometry collision box size=1.494866655312225 1 1; visual box size=1.494866655312225 1 1
- link rootLink000: geometry collision box size=1 1 1.567454954306859; visual box size=1 1 1.567454954306859
- link rootLink001: geometry collision box size=1.30324076016739 1 1; visual box size=1.30324076016739 1 1
- link rootLink01: geometry collision box size=1 1 1.3997647882262823; visual box size=1 1 1.3997647882262823
- link rootLink03: geometry collision box size=1 1.5493329004411809 1; visual box size=1 1.5493329004411809 1
Joints:
- removed joint rootLink0030_rootLink00300
- removed joint rootLink0030_rootLink00301
- removed joint rootLink0030_rootLink00304
- removed joint rootLink0031_rootLink00310
- removed joint rootLink0031_rootLink00311
- removed joint rootLink003_rootLink0030
- removed joint rootLink003_rootLink0031
- removed joint rootLink00_rootLink003
- removed joint rootLink01_rootLink010
- removed joint rootLink01_rootLink011
- added joint rootLink000_rootLink0000: type revolute, parent rootLink000, child rootLink0000, origin xyz=0 0.5 0.7837274771534295 rpy=0 0 0, axis 0 1 0, limit lower=-3.14159 upper=3.14159 effort=0.0 velocity=0.0
- added joint rootLink0010_rootLink00100: type revolute, parent rootLink0010, child rootLink00100, origin xyz=0 0 1.802701461242789 rpy=0 0 0, axis 0 0 1, limit lower=-3.14159 upper=3.14159 effort=0.0 velocity=0.0
- added joint rootLink0010_rootLink00101: type revolute, parent rootLink0010, child rootLink00101, origin xyz=0 0.5 0.9013507306213945 rpy=0 0 0, axis 1 0 0, limit lower=-3.14159 upper=3.14159 effort=0.0 velocity=0.0
- added joint rootLink001_rootLink0010: type revolute, parent rootLink001, child rootLink0010, origin xyz=0.651620380083695 0 0.5 rpy=0 0 0, axis 1 0 0, limit lower=-3.14159 upper=3.14159 effort=0.0 velocity=0.0
- added joint rootLink03_rootLink030: type revolute, parent rootLink03, child rootLink030, origin xyz=0.5 0.7746664502205904 0 rpy=0 0 0, axis 1 0 0, limit lower=-3.14159 upper=3.14159 effort=0.0 velocity=0.0
- added joint rootLink1002_rootLink10020: type revolute, parent rootLink1002, child rootLink10020, origin xyz=1.0910125194246736 0 0 rpy=0 0 0, axis 0 1 0, limit lower=-3.14159 upper=3.14159 effort=0.0 velocity=0.0
- added joint rootLink1002_rootLink10022: type revolute, parent rootLink1002, child rootLink10022, origin xyz=0.5455062597123368 0.5 0 rpy=0 0 0, axis 0 1 0, limit lower=-3.14159 upper=3.14159 effort=0.0 velocity=0.0
- added joint rootLink100_rootLink1000: type revolute, parent rootLink100, child rootLink1000, origin xyz=0 1.0813387183155512 0 rpy=0 0 0, axis 0 1 0, limit lower=-3.14159 upper=3.14159 effort=0.0 velocity=0.0
- added joint rootLink100_rootLink1002: type revolute, parent rootLink100, child rootLink1002, origin xyz=0.5 0.5406693591577756 0 rpy=0 0 0, axis 0 1 0, limit lower=-3.14159 upper=3.14159 effort=0.0 velocity=0.0
- added joint rootLink10_rootLink100: type revolute, parent rootLink10, child rootLink100, origin xyz=0.9441290297538336 0.5 0 rpy=0 0 0, axis 0 1 0, limit lower=-3.14159 upper=3.14159 effort=0.0 velocity=0.0
- added joint rootLink1_rootLink10: type revolute, parent rootLink1, child rootLink10, origin xyz=0.5 0 0.991029644343693 rpy=0 0 0, axis 0 0 1, limit lower=-3.14159 upper=3.14159 effort=0.0 velocity=0.0
- added joint rootLink1_rootLink12: type revolute, parent rootLink1, child rootLink12, origin xyz=0 0 1.982059288687386 rpy=0 0 0, axis 0 1 0, limit lower=-3.14159 upper=3.14159 effort=0.0 velocity=0.0
- added joint rootLink_rootLink1: type revolute, parent rootLink, child rootLink1, origin xyz=0 0 1.0 rpy=0 0 0, axis 0 0 1, limit lower=-3.14159 upper=3.14159 effort=0.0 velocity=0.0
- joint rootLink00_rootLink000: axis 0 1 0 -> 0 0 1; origin xyz=0 0 1.5872028841260102 rpy=0 0 0 -> xyz=0.7474333276561125 0 0.5 rpy=0 0 0
- joint rootLink00_rootLink001: axis 0 0 1 -> 0 1 0; origin xyz=0.5 0 0.7936014420630051 rpy=0 0 0 -> xyz=1.494866655312225 0 0 rpy=0 0 0
- joint rootLink0_rootLink00: axis 0 1 0 -> 1 0 0; origin xyz=0 0.8135001982699273 0.5 rpy=0 0 0 -> xyz=0.5 0.8702006159803533 0 rpy=0 0 0
- joint rootLink0_rootLink01: origin xyz=0.5 0.8135001982699273 0 rpy=0 0 0 -> xyz=0 0.8702006159803533 0.5 rpy=0 0 0
- joint rootLink0_rootLink03: axis 1 0 0 -> 0 1 0; origin xyz=0 1.6270003965398545 0 rpy=0 0 0 -> xyz=0 1.7404012319607065 0 rpy=0 0 0
- joint rootLink_rootLink0: axis 1 0 0 -> 0 0 1
