Commit message: final

File: bodies/body0.urdf (robot description, URDF)
Before this commit: robot robot, 1 links, 0 joints
Links:
- added link rootLink0, mass 1; collision box size=1 1 1.9844404494933823; visual box size=1 1 1.9844404494933823
- added link rootLink00, mass 1; collision box size=1.4130834853236505 1 1; visual box size=1.4130834853236505 1 1
- added link rootLink000, mass 1; collision box size=1.2541590407441887 1 1; visual box size=1.2541590407441887 1 1
- added link rootLink001, mass 1; collision box size=1 1.7044459296837995 1; visual box size=1 1.7044459296837995 1
Joints:
- added joint rootLink00_rootLink000: type revolute, parent rootLink00, child rootLink000, origin xyz=1.4130834853236505 0 0 rpy=0 0 0, axis 0 1 0, limit lower=-3.14159 upper=3.14159 effort=0.0 velocity=0.0
- added joint rootLink00_rootLink001: type revolute, parent rootLink00, child rootLink001, origin xyz=0.7065417426618252 0.5 0 rpy=0 0 0, axis 0 1 0, limit lower=-3.14159 upper=3.14159 effort=0.0 velocity=0.0
- added joint rootLink0_rootLink00: type revolute, parent rootLink0, child rootLink00, origin xyz=0.5 0 0.9922202247466911 rpy=0 0 0, axis 0 0 1, limit lower=-3.14159 upper=3.14159 effort=0.0 velocity=0.0
- added joint rootLink_rootLink0: type revolute, parent rootLink, child rootLink0, origin xyz=0 0 1.0 rpy=0 0 0, axis 0 1 0, limit lower=-3.14159 upper=3.14159 effort=0.0 velocity=0.0

File: bodies/body1.urdf (robot description, URDF)
Before this commit: robot robot, 6 links, 5 joints
Links:
- removed link rootLink01
- removed link rootLink010
- removed link rootLink011
- added link rootLink000, mass 1; collision box size=1.2541590407441887 1 1; visual box size=1.2541590407441887 1 1
- added link rootLink001, mass 1; collision box size=1 1.7044459296837995 1; visual box size=1 1.7044459296837995 1
- link rootLink0: geometry collision box size=1 1 1.9844404494933823; visual box size=1 1 1.9844404494933823
- link rootLink00: geometry collision box size=1.4130834853236505 1 1; visual box size=1.4130834853236505 1 1
Joints:
- removed joint rootLink01_rootLink010
- removed joint rootLink01_rootLink011
- removed joint rootLink0_rootLink01
- added joint rootLink00_rootLink000: type revolute, parent rootLink00, child rootLink000, origin xyz=1.4130834853236505 0 0 rpy=0 0 0, axis 0 1 0, limit lower=-3.14159 upper=3.14159 effort=0.0 velocity=0.0
- added joint rootLink00_rootLink001: type revolute, parent rootLink00, child rootLink001, origin xyz=0.7065417426618252 0.5 0 rpy=0 0 0, axis 0 1 0, limit lower=-3.14159 upper=3.14159 effort=0.0 velocity=0.0
- joint rootLink0_rootLink00: origin xyz=0 -0.5 0.6320906100443943 rpy=0 0 0 -> xyz=0.5 0 0.9922202247466911 rpy=0 0 0
- joint rootLink_rootLink0: axis 1 0 0 -> 0 1 0

File: bodies/body100.urdf (robot description, URDF)
Before this commit: robot robot, 1 links, 0 joints
Links:
- added link rootLink0, mass 1; collision box size=1 1 1.3605562588676265; visual box size=1 1 1.3605562588676265
- added link rootLink01, mass 1; collision box size=1.2087311436275017 1 1; visual box size=1.2087311436275017 1 1
Joints:
- added joint rootLink0_rootLink01: type revolute, parent rootLink0, child rootLink01, origin xyz=-0.5 0 0.6802781294338133 rpy=0 0 0, axis 0 1 0, limit lower=-3.14159 upper=3.14159 effort=0.0 velocity=0.0
- added joint rootLink_rootLink0: type revolute, parent rootLink, child rootLink0, origin xyz=0 0 1.0 rpy=0 0 0, axis 1 0 0, limit lower=-3.14159 upper=3.14159 effort=0.0 velocity=0.0

File: bodies/body101.urdf (robot description, URDF)
Before this commit: robot robot, 6 links, 5 joints
Links:
- removed link rootLink00
- removed link rootLink010
- removed link rootLink011
- link rootLink0: geometry collision box size=1 1 1.3605562588676265; visual box size=1 1 1.3605562588676265
- link rootLink01: geometry collision box size=1.2087311436275017 1 1; visual box size=1.2087311436275017 1 1
Joints:
- removed joint rootLink01_rootLink010
- removed joint rootLink01_rootLink011
- removed joint rootLink0_rootLink00
- joint rootLink0_rootLink01: origin xyz=-0.5 0 0.6320906100443943 rpy=0 0 0 -> xyz=-0.5 0 0.6802781294338133 rpy=0 0 0

File: bodies/body102.urdf (robot description, URDF)
Before this commit: robot robot, 1 links, 0 joints
Links:
- added link rootLink0, mass 1; collision box size=1 1 1.3605562588676265; visual box size=1 1 1.3605562588676265
- added link rootLink01, mass 1; collision box size=1.2087311436275017 1 1; visual box size=1.2087311436275017 1 1
Joints:
- added joint rootLink0_rootLink01: type revolute, parent rootLink0, child rootLink01, origin xyz=-0.5 0 0.6802781294338133 rpy=0 0 0, axis 0 1 0, limit lower=-3.14159 upper=3.14159 effort=0.0 velocity=0.0
- added joint rootLink_rootLink0: type revolute, parent rootLink, child rootLink0, origin xyz=0 0 1.0 rpy=0 0 0, axis 1 0 0, limit lower=-3.14159 upper=3.14159 effort=0.0 velocity=0.0

File: bodies/body103.urdf (robot description, URDF)
Before this commit: robot robot, 6 links, 5 joints
Links:
- removed link rootLink1
- removed link rootLink10
- removed link rootLink100
- removed link rootLink1000
- removed link rootLink11
- added link rootLink0, mass 1; collision box size=1 1 1.3605562588676265; visual box size=1 1 1.3605562588676265
- added link rootLink01, mass 1; collision box size=1.2087311436275017 1 1; visual box size=1.2087311436275017 1 1
Joints:
- removed joint rootLink100_rootLink1000
- removed joint rootLink10_rootLink100
- removed joint rootLink1_rootLink10
- removed joint rootLink1_rootLink11
- removed joint rootLink_rootLink1
- added joint rootLink0_rootLink01: type revolute, parent rootLink0, child rootLink01, origin xyz=-0.5 0 0.6802781294338133 rpy=0 0 0, axis 0 1 0, limit lower=-3.14159 upper=3.14159 effort=0.0 velocity=0.0
- added joint rootLink_rootLink0: type revolute, parent rootLink, child rootLink0, origin xyz=0 0 1.0 rpy=0 0 0, axis 1 0 0, limit lower=-3.14159 upper=3.14159 effort=0.0 velocity=0.0

File: bodies/body105.urdf (robot description, URDF)
Before this commit: robot robot, 31 links, 30 joints
Links:
- removed link rootLink00
- removed link rootLink000
- removed link rootLink0000
- removed link rootLink00001
- removed link rootLink000010
- removed link rootLink001
- removed link rootLink0010
- removed link rootLink0011
- removed link rootLink00110
- removed link rootLink00111
- removed link rootLink00113
- removed link rootLink001130
- removed link rootLink001131
- removed link rootLink002
- removed link rootLink0020
- removed link rootLink00200
- removed link rootLink010
- removed link rootLink0101
- removed link rootLink01010
- removed link rootLink011
- removed link rootLink013
- removed link rootLink0130
- removed link rootLink01300
- removed link rootLink013001
- removed link rootLink0130010
- removed link rootLink0130012
- removed link rootLink01303
- removed link rootLink0131
- link rootLink0: geometry collision box size=1 1 1.3605562588676265; visual box size=1 1 1.3605562588676265
- link rootLink01: geometry collision box size=1.2087311436275017 1 1; visual box size=1.2087311436275017 1 1
Joints:
- removed joint rootLink00001_rootLink000010
- removed joint rootLink0000_rootLink00001
- removed joint rootLink000_rootLink0000
- removed joint rootLink00113_rootLink001130
- removed joint rootLink00113_rootLink001131
- removed joint rootLink0011_rootLink00110
- removed joint rootLink0011_rootLink00111
- removed joint rootLink0011_rootLink00113
- removed joint rootLink001_rootLink0010
- removed joint rootLink001_rootLink0011
- removed joint rootLink0020_rootLink00200
- removed joint rootLink002_rootLink0020
- removed joint rootLink00_rootLink000
- removed joint rootLink00_rootLink001
- removed joint rootLink00_rootLink002
- removed joint rootLink0101_rootLink01010
- removed joint rootLink010_rootLink0101
- removed joint rootLink013001_rootLink0130010
- removed joint rootLink013001_rootLink0130012
- removed joint rootLink01300_rootLink013001
- removed joint rootLink0130_rootLink01300
- removed joint rootLink0130_rootLink01303
- removed joint rootLink013_rootLink0130
- removed joint rootLink013_rootLink0131
- removed joint rootLink01_rootLink010
- removed joint rootLink01_rootLink011
- removed joint rootLink01_rootLink013
- removed joint rootLink0_rootLink00
- joint rootLink0_rootLink01: axis 1 0 0 -> 0 1 0; origin xyz=-0.5 0 0.5231012439279966 rpy=0 0 0 -> xyz=-0.5 0 0.6802781294338133 rpy=0 0 0
- joint rootLink_rootLink0: axis 0 0 1 -> 1 0 0

File: bodies/body106.urdf (robot description, URDF)
Before this commit: robot robot, 10 links, 9 joints
Links:
- removed link rootLink00
- removed link rootLink002
- removed link rootLink0020
- removed link rootLink00200
- removed link rootLink00201
- removed link rootLink0021
- removed link rootLink010
- link rootLink0: geometry collision box size=1 1 1.3605562588676265; visual box size=1 1 1.3605562588676265
- link rootLink01: geometry collision box size=1.2087311436275017 1 1; visual box size=1.2087311436275017 1 1
Joints:
- removed joint rootLink0020_rootLink00200
- removed joint rootLink0020_rootLink00201
- removed joint rootLink002_rootLink0020
- removed joint rootLink002_rootLink0021
- removed joint rootLink00_rootLink002
- removed joint rootLink01_rootLink010
- removed joint rootLink0_rootLink00
- joint rootLink0_rootLink01: axis 1 0 0 -> 0 1 0; origin xyz=-0.5 0 0.5100670244117298 rpy=0 0 0 -> xyz=-0.5 0 0.6802781294338133 rpy=0 0 0
- joint rootLink_rootLink0: axis 0 1 0 -> 1 0 0

File: bodies/body107.urdf (robot description, URDF)
Before this commit: robot robot, 8 links, 7 joints
Links:
- removed link rootLink1
- removed link rootLink10
- removed link rootLink100
- removed link rootLink1001
- removed link rootLink10010
- removed link rootLink100100
- removed link rootLink1002
- added link rootLink0, mass 1; collision box size=1 1 1.3605562588676265; visual box size=1 1 1.3605562588676265
- added link rootLink01, mass 1; collision box size=1.2087311436275017 1 1; visual box size=1.2087311436275017 1 1
Joints:
- removed joint rootLink10010_rootLink100100
- removed joint rootLink1001_rootLink10010
- removed joint rootLink100_rootLink1001
- removed joint rootLink100_rootLink1002
- removed joint rootLink10_rootLink100
- removed joint rootLink1_rootLink10
- removed joint rootLink_rootLink1
- added joint rootLink0_rootLink01: type revolute, parent rootLink0, child rootLink01, origin xyz=-0.5 0 0.6802781294338133 rpy=0 0 0, axis 0 1 0, limit lower=-3.14159 upper=3.14159 effort=0.0 velocity=0.0
- added joint rootLink_rootLink0: type revolute, parent rootLink, child rootLink0, origin xyz=0 0 1.0 rpy=0 0 0, axis 1 0 0, limit lower=-3.14159 upper=3.14159 effort=0.0 velocity=0.0

File: bodies/body111.urdf (robot description, URDF)
Before this commit: robot robot, 14 links, 13 joints
Links:
- removed link rootLink00
- removed link rootLink000
- removed link rootLink0000
- removed link rootLink0001
- removed link rootLink02
- removed link rootLink020
- removed link rootLink0200
- removed link rootLink0202
- removed link rootLink02020
- removed link rootLink022
- removed link rootLink0220
- removed link rootLink03
- added link rootLink01, mass 1; collision box size=1.2087311436275017 1 1; visual box size=1.2087311436275017 1 1
- link rootLink0: geometry collision box size=1 1 1.3605562588676265; visual box size=1 1 1.3605562588676265
Joints:
- removed joint rootLink000_rootLink0000
- removed joint rootLink000_rootLink0001
- removed joint rootLink00_rootLink000
- removed joint rootLink0202_rootLink02020
- removed joint rootLink020_rootLink0200
- removed joint rootLink020_rootLink0202
- removed joint rootLink022_rootLink0220
- removed joint rootLink02_rootLink020
- removed joint rootLink02_rootLink022
- removed joint rootLink0_rootLink00
- removed joint rootLink0_rootLink02
- removed joint rootLink0_rootLink03
- added joint rootLink0_rootLink01: type revolute, parent rootLink0, child rootLink01, origin xyz=-0.5 0 0.6802781294338133 rpy=0 0 0, axis 0 1 0, limit lower=-3.14159 upper=3.14159 effort=0.0 velocity=0.0

File: bodies/body114.urdf (robot description, URDF)
Before this commit: robot robot, 8 links, 7 joints
Links:
- removed link rootLink00
- removed link rootLink000
- removed link rootLink0000
- removed link rootLink00000
- removed link rootLink000001
- removed link rootLink0002
- added link rootLink01, mass 1; collision box size=1.2087311436275017 1 1; visual box size=1.2087311436275017 1 1
- link rootLink0: geometry collision box size=1 1 1.3605562588676265; visual box size=1 1 1.3605562588676265
Joints:
- removed joint rootLink00000_rootLink000001
- removed joint rootLink0000_rootLink00000
- removed joint rootLink000_rootLink0000
- removed joint rootLink000_rootLink0002
- removed joint rootLink00_rootLink000
- removed joint rootLink0_rootLink00
- added joint rootLink0_rootLink01: type revolute, parent rootLink0, child rootLink01, origin xyz=-0.5 0 0.6802781294338133 rpy=0 0 0, axis 0 1 0, limit lower=-3.14159 upper=3.14159 effort=0.0 velocity=0.0
- joint rootLink_rootLink0: axis 0 1 0 -> 1 0 0

File: bodies/body120.urdf (robot description, URDF)
Before this commit: robot robot, 1 links, 0 joints
Links:
- added link rootLink0, mass 1; collision box size=1 1 1.6660715157316761; visual box size=1 1 1.6660715157316761
- added link rootLink00, mass 1; collision box size=1.1415739418915365 1 1; visual box size=1.1415739418915365 1 1
- added link rootLink000, mass 1; collision box size=1 1.7339678888251595 1; visual box size=1 1.7339678888251595 1
- added link rootLink0000, mass 1; collision box size=1.2405647372978112 1 1; visual box size=1.2405647372978112 1 1
Joints:
- added joint rootLink000_rootLink0000: type revolute, parent rootLink000, child rootLink0000, origin xyz=0.5 0.8669839444125798 0 rpy=0 0 0, axis 0 0 1, limit lower=-3.14159 upper=3.14159 effort=0.0 velocity=0.0
- added joint rootLink00_rootLink000: type revolute, parent rootLink00, child rootLink000, origin xyz=0.5707869709457682 0.5 0 rpy=0 0 0, axis 0 1 0, limit lower=-3.14159 upper=3.14159 effort=0.0 velocity=0.0
- added joint rootLink0_rootLink00: type revolute, parent rootLink0, child rootLink00, origin xyz=0.5 0 0.8330357578658381 rpy=0 0 0, axis 0 1 0, limit lower=-3.14159 upper=3.14159 effort=0.0 velocity=0.0
- added joint rootLink_rootLink0: type revolute, parent rootLink, child rootLink0, origin xyz=0 0 1.0 rpy=0 0 0, axis 0 1 0, limit lower=-3.14159 upper=3.14159 effort=0.0 velocity=0.0

File: bodies/body121.urdf (robot description, URDF)
Before this commit: robot robot, 1 links, 0 joints
Links:
- added link rootLink0, mass 1; collision box size=1 1 1.6660715157316761; visual box size=1 1 1.6660715157316761
- added link rootLink00, mass 1; collision box size=1.1415739418915365 1 1; visual box size=1.1415739418915365 1 1
- added link rootLink000, mass 1; collision box size=1 1.7339678888251595 1; visual box size=1 1.7339678888251595 1
- added link rootLink0000, mass 1; collision box size=1.2405647372978112 1 1; visual box size=1.2405647372978112 1 1
Joints:
- added joint rootLink000_rootLink0000: type revolute, parent rootLink000, child rootLink0000, origin xyz=0.5 0.8669839444125798 0 rpy=0 0 0, axis 0 0 1, limit lower=-3.14159 upper=3.14159 effort=0.0 velocity=0.0
- added joint rootLink00_rootLink000: type revolute, parent rootLink00, child rootLink000, origin xyz=0.5707869709457682 0.5 0 rpy=0 0 0, axis 0 1 0, limit lower=-3.14159 upper=3.14159 effort=0.0 velocity=0.0
- added joint rootLink0_rootLink00: type revolute, parent rootLink0, child rootLink00, origin xyz=0.5 0 0.8330357578658381 rpy=0 0 0, axis 0 1 0, limit lower=-3.14159 upper=3.14159 effort=0.0 velocity=0.0
- added joint rootLink_rootLink0: type revolute, parent rootLink, child rootLink0, origin xyz=0 0 1.0 rpy=0 0 0, axis 0 1 0, limit lower=-3.14159 upper=3.14159 effort=0.0 velocity=0.0

File: bodies/body122.urdf (robot description, URDF)
Before this commit: robot robot, 9 links, 8 joints
Links:
- removed link rootLink4
- removed link rootLink41
- removed link rootLink410
- removed link rootLink4101
- removed link rootLink41010
- removed link rootLink410100
- removed link rootLink4101000
- removed link rootLink4101001
- added link rootLink0, mass 1; collision box size=1 1 1.6660715157316761; visual box size=1 1 1.6660715157316761
- added link rootLink00, mass 1; collision box size=1.1415739418915365 1 1; visual box size=1.1415739418915365 1 1
- added link rootLink000, mass 1; collision box size=1 1.7339678888251595 1; visual box size=1 1.7339678888251595 1
- added link rootLink0000, mass 1; collision box size=1.2405647372978112 1 1; visual box size=1.2405647372978112 1 1
Joints:
- removed joint rootLink410100_rootLink4101000
- removed joint rootLink410100_rootLink4101001
- removed joint rootLink41010_rootLink410100
- removed joint rootLink4101_rootLink41010
- removed joint rootLink410_rootLink4101
- removed joint rootLink41_rootLink410
- removed joint rootLink4_rootLink41
- removed joint rootLink_rootLink4
- added joint rootLink000_rootLink0000: type revolute, parent rootLink000, child rootLink0000, origin xyz=0.5 0.8669839444125798 0 rpy=0 0 0, axis 0 0 1, limit lower=-3.14159 upper=3.14159 effort=0.0 velocity=0.0
- added joint rootLink00_rootLink000: type revolute, parent rootLink00, child rootLink000, origin xyz=0.5707869709457682 0.5 0 rpy=0 0 0, axis 0 1 0, limit lower=-3.14159 upper=3.14159 effort=0.0 velocity=0.0
- added joint rootLink0_rootLink00: type revolute, parent rootLink0, child rootLink00, origin xyz=0.5 0 0.8330357578658381 rpy=0 0 0, axis 0 1 0, limit lower=-3.14159 upper=3.14159 effort=0.0 velocity=0.0
- added joint rootLink_rootLink0: type revolute, parent rootLink, child rootLink0, origin xyz=0 0 1.0 rpy=0 0 0, axis 0 1 0, limit lower=-3.14159 upper=3.14159 effort=0.0 velocity=0.0

File: bodies/body132.urdf (robot description, URDF)
Before this commit: robot robot, 8 links, 7 joints
Links:
- removed link rootLink2
- removed link rootLink22
- removed link rootLink221
- removed link rootLink2210
- removed link rootLink2211
- removed link rootLink22110
- removed link rootLink22112
- added link rootLink0, mass 1; collision box size=1 1 1.6660715157316761; visual box size=1 1 1.6660715157316761
- added link rootLink00, mass 1; collision box size=1.1415739418915365 1 1; visual box size=1.1415739418915365 1 1
- added link rootLink000, mass 1; collision box size=1 1.7339678888251595 1; visual box size=1 1.7339678888251595 1
- added link rootLink0000, mass 1; collision box size=1.2405647372978112 1 1; visual box size=1.2405647372978112 1 1
Joints:
- removed joint rootLink2211_rootLink22110
- removed joint rootLink2211_rootLink22112
- removed joint rootLink221_rootLink2210
- removed joint rootLink221_rootLink2211
- removed joint rootLink22_rootLink221
- removed joint rootLink2_rootLink22
- removed joint rootLink_rootLink2
- added joint rootLink000_rootLink0000: type revolute, parent rootLink000, child rootLink0000, origin xyz=0.5 0.8669839444125798 0 rpy=0 0 0, axis 0 0 1, limit lower=-3.14159 upper=3.14159 effort=0.0 velocity=0.0
- added joint rootLink00_rootLink000: type revolute, parent rootLink00, child rootLink000, origin xyz=0.5707869709457682 0.5 0 rpy=0 0 0, axis 0 1 0, limit lower=-3.14159 upper=3.14159 effort=0.0 velocity=0.0
- added joint rootLink0_rootLink00: type revolute, parent rootLink0, child rootLink00, origin xyz=0.5 0 0.8330357578658381 rpy=0 0 0, axis 0 1 0, limit lower=-3.14159 upper=3.14159 effort=0.0 velocity=0.0
- added joint rootLink_rootLink0: type revolute, parent rootLink, child rootLink0, origin xyz=0 0 1.0 rpy=0 0 0, axis 0 1 0, limit lower=-3.14159 upper=3.14159 effort=0.0 velocity=0.0

File: bodies/body133.urdf (robot description, URDF)
Before this commit: robot robot, 15 links, 14 joints
Links:
- removed link rootLink0001
- removed link rootLink00010
- removed link rootLink003
- removed link rootLink0030
- removed link rootLink0031
- removed link rootLink00310
- removed link rootLink004
- removed link rootLink0041
- removed link rootLink00410
- removed link rootLink004101
- removed link rootLink00412
- added link rootLink0000, mass 1; collision box size=1.2405647372978112 1 1; visual box size=1.2405647372978112 1 1
- link rootLink0: geometry collision box size=1 1 1.6660715157316761; visual box size=1 1 1.6660715157316761
- link rootLink00: geometry collision box size=1.1415739418915365 1 1; visual box size=1.1415739418915365 1 1
- link rootLink000: geometry collision box size=1 1.7339678888251595 1; visual box size=1 1.7339678888251595 1
Joints:
- removed joint rootLink0001_rootLink00010
- removed joint rootLink000_rootLink0001
- removed joint rootLink0031_rootLink00310
- removed joint rootLink003_rootLink0030
- removed joint rootLink003_rootLink0031
- removed joint rootLink00410_rootLink004101
- removed joint rootLink0041_rootLink00410
- removed joint rootLink0041_rootLink00412
- removed joint rootLink004_rootLink0041
- removed joint rootLink00_rootLink003
- removed joint rootLink00_rootLink004
- added joint rootLink000_rootLink0000: type revolute, parent rootLink000, child rootLink0000, origin xyz=0.5 0.8669839444125798 0 rpy=0 0 0, axis 0 0 1, limit lower=-3.14159 upper=3.14159 effort=0.0 velocity=0.0
- joint rootLink00_rootLink000: axis 1 0 0 -> 0 1 0; origin xyz=1.7666354598146765 0 0 rpy=0 0 0 -> xyz=0.5707869709457682 0.5 0 rpy=0 0 0
- joint rootLink0_rootLink00: axis 0 0 1 -> 0 1 0; origin xyz=0.5 0 0.928556336909977 rpy=0 0 0 -> xyz=0.5 0 0.8330357578658381 rpy=0 0 0
