Commit message: final

File: bodies/body140.urdf (robot description, URDF)
Before this commit: robot robot, 25 links, 24 joints
Links:
- removed link rootLink1
- removed link rootLink10
- removed link rootLink100
- removed link rootLink1000
- removed link rootLink11
- removed link rootLink110
- removed link rootLink1100
- removed link rootLink11001
- removed link rootLink110010
- removed link rootLink1100100
- removed link rootLink110012
- removed link rootLink1101
- removed link rootLink11010
- removed link rootLink110100
- removed link rootLink110101
- removed link rootLink11012
- removed link rootLink110120
- removed link rootLink1101200
- removed link rootLink11012000
- removed link rootLink11012001
- removed link rootLink1101201
- removed link rootLink12
- removed link rootLink120
- removed link rootLink1200
- added link rootLink4, mass 1; collision box size=1 1 1.7027907029787666; visual box size=1 1 1.7027907029787666
- added link rootLink40, mass 1; collision box size=1 1.3398928529683745 1; visual box size=1 1.3398928529683745 1
- added link rootLink400, mass 1; collision box size=1 1 1.4730742657893083; visual box size=1 1 1.4730742657893083
Joints:
- removed joint rootLink100_rootLink1000
- removed joint rootLink10_rootLink100
- removed joint rootLink110010_rootLink1100100
- removed joint rootLink11001_rootLink110010
- removed joint rootLink11001_rootLink110012
- removed joint rootLink1100_rootLink11001
- removed joint rootLink11010_rootLink110100
- removed joint rootLink11010_rootLink110101
- removed joint rootLink1101200_rootLink11012000
- removed joint rootLink1101200_rootLink11012001
- removed joint rootLink110120_rootLink1101200
- removed joint rootLink110120_rootLink1101201
- removed joint rootLink11012_rootLink110120
- removed joint rootLink1101_rootLink11010
- removed joint rootLink1101_rootLink11012
- removed joint rootLink110_rootLink1100
- removed joint rootLink110_rootLink1101
- removed joint rootLink11_rootLink110
- removed joint rootLink120_rootLink1200
- removed joint rootLink12_rootLink120
- removed joint rootLink1_rootLink10
- removed joint rootLink1_rootLink11
- removed joint rootLink1_rootLink12
- removed joint rootLink_rootLink1
- added joint rootLink40_rootLink400: type revolute, parent rootLink40, child rootLink400, origin xyz=0 -0.6699464264841872 0.5 rpy=0 0 0, axis 1 0 0, limit lower=-3.14159 upper=3.14159 effort=0.0 velocity=0.0
- added joint rootLink4_rootLink40: type revolute, parent rootLink4, child rootLink40, origin xyz=0 -0.5 0.8513953514893833 rpy=0 0 0, axis 1 0 0, limit lower=-3.14159 upper=3.14159 effort=0.0 velocity=0.0
- added joint rootLink_rootLink4: type revolute, parent rootLink, child rootLink4, origin xyz=0 0 1.0 rpy=0 0 0, axis 1 0 0, limit lower=-3.14159 upper=3.14159 effort=0.0 velocity=0.0

File: bodies/body141.urdf (robot description, URDF)
Before this commit: robot robot, 1 links, 0 joints
Links:
- added link rootLink4, mass 1; collision box size=1 1 1.7027907029787666; visual box size=1 1 1.7027907029787666
- added link rootLink40, mass 1; collision box size=1 1.3398928529683745 1; visual box size=1 1.3398928529683745 1
- added link rootLink400, mass 1; collision box size=1 1 1.4730742657893083; visual box size=1 1 1.4730742657893083
Joints:
- added joint rootLink40_rootLink400: type revolute, parent rootLink40, child rootLink400, origin xyz=0 -0.6699464264841872 0.5 rpy=0 0 0, axis 1 0 0, limit lower=-3.14159 upper=3.14159 effort=0.0 velocity=0.0
- added joint rootLink4_rootLink40: type revolute, parent rootLink4, child rootLink40, origin xyz=0 -0.5 0.8513953514893833 rpy=0 0 0, axis 1 0 0, limit lower=-3.14159 upper=3.14159 effort=0.0 velocity=0.0
- added joint rootLink_rootLink4: type revolute, parent rootLink, child rootLink4, origin xyz=0 0 1.0 rpy=0 0 0, axis 1 0 0, limit lower=-3.14159 upper=3.14159 effort=0.0 velocity=0.0

File: bodies/body142.urdf (robot description, URDF)
Before this commit: robot robot, 9 links, 8 joints
Links:
- removed link rootLink2
- removed link rootLink20
- removed link rootLink202
- removed link rootLink2021
- removed link rootLink2024
- removed link rootLink21
- removed link rootLink210
- removed link rootLink2100
- added link rootLink4, mass 1; collision box size=1 1 1.7027907029787666; visual box size=1 1 1.7027907029787666
- added link rootLink40, mass 1; collision box size=1 1.3398928529683745 1; visual box size=1 1.3398928529683745 1
- added link rootLink400, mass 1; collision box size=1 1 1.4730742657893083; visual box size=1 1 1.4730742657893083
Joints:
- removed joint rootLink202_rootLink2021
- removed joint rootLink202_rootLink2024
- removed joint rootLink20_rootLink202
- removed joint rootLink210_rootLink2100
- removed joint rootLink21_rootLink210
- removed joint rootLink2_rootLink20
- removed joint rootLink2_rootLink21
- removed joint rootLink_rootLink2
- added joint rootLink40_rootLink400: type revolute, parent rootLink40, child rootLink400, origin xyz=0 -0.6699464264841872 0.5 rpy=0 0 0, axis 1 0 0, limit lower=-3.14159 upper=3.14159 effort=0.0 velocity=0.0
- added joint rootLink4_rootLink40: type revolute, parent rootLink4, child rootLink40, origin xyz=0 -0.5 0.8513953514893833 rpy=0 0 0, axis 1 0 0, limit lower=-3.14159 upper=3.14159 effort=0.0 velocity=0.0
- added joint rootLink_rootLink4: type revolute, parent rootLink, child rootLink4, origin xyz=0 0 1.0 rpy=0 0 0, axis 1 0 0, limit lower=-3.14159 upper=3.14159 effort=0.0 velocity=0.0

File: bodies/body143.urdf (robot description, URDF)
Before this commit: robot robot, 5 links, 4 joints
Links:
- removed link rootLink0
- removed link rootLink00
- removed link rootLink000
- removed link rootLink0000
- added link rootLink4, mass 1; collision box size=1 1 1.7027907029787666; visual box size=1 1 1.7027907029787666
- added link rootLink40, mass 1; collision box size=1 1.3398928529683745 1; visual box size=1 1.3398928529683745 1
- added link rootLink400, mass 1; collision box size=1 1 1.4730742657893083; visual box size=1 1 1.4730742657893083
Joints:
- removed joint rootLink000_rootLink0000
- removed joint rootLink00_rootLink000
- removed joint rootLink0_rootLink00
- removed joint rootLink_rootLink0
- added joint rootLink40_rootLink400: type revolute, parent rootLink40, child rootLink400, origin xyz=0 -0.6699464264841872 0.5 rpy=0 0 0, axis 1 0 0, limit lower=-3.14159 upper=3.14159 effort=0.0 velocity=0.0
- added joint rootLink4_rootLink40: type revolute, parent rootLink4, child rootLink40, origin xyz=0 -0.5 0.8513953514893833 rpy=0 0 0, axis 1 0 0, limit lower=-3.14159 upper=3.14159 effort=0.0 velocity=0.0
- added joint rootLink_rootLink4: type revolute, parent rootLink, child rootLink4, origin xyz=0 0 1.0 rpy=0 0 0, axis 1 0 0, limit lower=-3.14159 upper=3.14159 effort=0.0 velocity=0.0
